Commit message: introduced upperarm and forearm

File: ros2_ws/src/human_arm_model/urdf/model.urdf.xacro (robot description, xacro)
@@ -13,3 +13,28 @@
         </visual>
     </link>
+    <joint name="shoulder_joint" type="continuous">
+        <parent link="torso"/>
+        <child link="upperarm"/>
+        <origin xyz="0.5 0 0.5"/>
+    </joint>
+    <link name="upperarm">
+        <visual>
+            <geometry>
+                <cylinder length="${upperarm_length}" radius="${upperarm_circumference/ (2* math.pi)}"/>
+            </geometry>
+            <origin xyz="${upperarm_length/2} 0 0" rpy="0 ${math.pi/2} 0" />
+        </visual>
+    </link>
+    <joint name="elbow_joint" type="continuous">
+        <parent link="upperarm"/>
+        <child link="forearm"/>
+        <origin xyz="${upperarm_length} 0 0"/>
+    </joint>
+    <link name="forearm">
+        <visual>
+            <geometry>
+                <cylinder length="${elbow_wrist_length}" radius="${forearm_circumference / (2*math.pi)}" />
+            </geometry>
+        </visual>
+    </link>
 </robot>

Commit message: Model with working limits for shoulder and elbow movement created; values for those limits are to be changend

File: ros2_ws/src/human_arm_model/urdf/model.urdf.xacro (robot description, xacro)
@@ -9,13 +9,38 @@
         <visual>
             <geometry>
-                <box size="1.0 1.0 1.0"/>
+                <box size="1.0 ${0.2+ upperarm_circumference/ (2* math.pi)} 1.0"/>
             </geometry>
         </visual>
     </link>
-    <joint name="shoulder_joint" type="continuous">
-        <parent link="torso"/>
-        <child link="upperarm"/>
+    <!-- ___________________ Shoulder joint __________ -->
+    <xacro:macro name="shoulder_template" params="suffix parent child:='' *origin *axis *limit">
+        <joint name="shoulder_${suffix}_joint" type="revolute">
+            <parent link="${parent if parent == 'torso' else 'shoulder_'+parent+'_link'}"/>
+            <child link="${child if child != '' else 'shoulder_' + suffix + '_link'}"/>
+            <xacro:insert_block name="origin"/>
+            <xacro:insert_block name="axis"/>
+            <xacro:insert_block name="limit"/>
+        </joint>
+        <xacro:if value="${child == ''}">
+            <link name="shoulder_${suffix}_link">
+            </link>
+        </xacro:if>
+    </xacro:macro>
+    <xacro:shoulder_template suffix="yaw" parent="torso">
         <origin xyz="0.5 0 0.5"/>
-    </joint>
+        <axis xyz="0 -1 0" />
+        <limit effort="1000" lower="-1.1" upper="1.9" velocity="0.5" />
+    </xacro:shoulder_template>
+    <xacro:shoulder_template suffix="pitch" parent="yaw">
+        <origin xyz="0 0 0"/>
+        <axis xyz="0 0 1"/>
+        <limit effort="1000" lower="-0.4" upper="3.3" velocity="0.5" />
+    </xacro:shoulder_template>
+    <xacro:shoulder_template suffix="roll" parent="pitch" child="upperarm">
+        <origin xyz="0 0 0"/>
+        <axis xyz="1 0 0"/>
+        <!-- Bullshit limit for now  -->
+        <limit effort="1000" lower="-0.4" upper="3.3" velocity="0.5" />
+    </xacro:shoulder_template>
     <link name="upperarm">
         <visual>
@@ -26,7 +51,10 @@
         </visual>
     </link>
-    <joint name="elbow_joint" type="continuous">
+    <!-- ____________________ Elbow joint ___________ -->
+    <joint name="elbow_joint" type="revolute">
         <parent link="upperarm"/>
         <child link="forearm"/>
+        <axis xyz="0 0 1" />
+        <limit effort="1000" lower="0" upper="2.5" velocity="0.5" />
         <origin xyz="${upperarm_length} 0 0"/>
     </joint>
@@ -36,4 +64,5 @@
                 <cylinder length="${elbow_wrist_length}" radius="${forearm_circumference / (2*math.pi)}" />
             </geometry>
+            <origin xyz="${elbow_wrist_length/2} 0 0" rpy="0 ${math.pi/2} 0"/>
         </visual>
     </link>

Commit message: further abstraction in macro for reuse in elbow joint

File: ros2_ws/src/human_arm_model/urdf/model.urdf.xacro (robot description, xacro)
@@ -14,8 +14,8 @@
     </link>
     <!-- ___________________ Shoulder joint __________ -->
-    <xacro:macro name="shoulder_template" params="suffix parent child:='' *origin *axis *limit">
-        <joint name="shoulder_${suffix}_joint" type="revolute">
-            <parent link="${parent if parent == 'torso' else 'shoulder_'+parent+'_link'}"/>
-            <child link="${child if child != '' else 'shoulder_' + suffix + '_link'}"/>
+    <xacro:macro name="shoulder_template" params="bodypart suffix parent child:='' *origin *axis *limit">
+        <joint name="${bodypart}_${suffix}_joint" type="revolute">
+            <parent link="${parent if parent == 'torso' else bodypart+'_'+parent+'_link'}"/>
+            <child link="${child if child != '' else bodypart+'_' + suffix + '_link'}"/>
             <xacro:insert_block name="origin"/>
             <xacro:insert_block name="axis"/>
@@ -23,19 +23,19 @@
         </joint>
         <xacro:if value="${child == ''}">
-            <link name="shoulder_${suffix}_link">
+            <link name="${bodypart}_${suffix}_link">
             </link>
         </xacro:if>
     </xacro:macro>
-    <xacro:shoulder_template suffix="yaw" parent="torso">
+    <xacro:shoulder_template bodypart="shoulder" suffix="yaw" parent="torso">
         <origin xyz="0.5 0 0.5"/>
         <axis xyz="0 -1 0" />
         <limit effort="1000" lower="-1.1" upper="1.9" velocity="0.5" />
     </xacro:shoulder_template>
-    <xacro:shoulder_template suffix="pitch" parent="yaw">
+    <xacro:shoulder_template bodypart="shoulder" suffix="pitch" parent="yaw">
         <origin xyz="0 0 0"/>
         <axis xyz="0 0 1"/>
         <limit effort="1000" lower="-0.4" upper="3.3" velocity="0.5" />
     </xacro:shoulder_template>
-    <xacro:shoulder_template suffix="roll" parent="pitch" child="upperarm">
+    <xacro:shoulder_template bodypart="shoulder" suffix="roll" parent="pitch" child="upperarm">
         <origin xyz="0 0 0"/>
         <axis xyz="1 0 0"/>

Commit message: put constants in seperate file & added both wrist and can

File: ros2_ws/src/human_arm_model/urdf/model.urdf.xacro (robot description, xacro)
@@ -1,12 +1,9 @@
 <?xml version="1.0"?>
 <robot xmlns:xacro="http://www.ros.org/wiki/xacro" name="human_arm_modell">
-    <xacro:property name="upperarm_length" value="0.3637"/>
-    <xacro:property name="elbow_wrist_length" value="0.2869"/>
-    <xacro:property name="upperarm_circumference" value="0.3581"/>
-    <xacro:property name="wrist_circumference" value="0.1759"/>
-    <xacro:property name="forearm_circumference" value="0.3101"/>
+    <xacro:include filename="constants.urdf.xacro" />
     <link name="torso">
         <visual>
             <geometry>
+                <!-- Bullshit limit for now  -->
                 <box size="1.0 ${0.2+ upperarm_circumference/ (2* math.pi)} 1.0"/>
             </geometry>
@@ -14,33 +11,20 @@
     </link>
     <!-- ___________________ Shoulder joint __________ -->
-    <xacro:macro name="shoulder_template" params="bodypart suffix parent child:='' *origin *axis *limit">
-        <joint name="${bodypart}_${suffix}_joint" type="revolute">
-            <parent link="${parent if parent == 'torso' else bodypart+'_'+parent+'_link'}"/>
-            <child link="${child if child != '' else bodypart+'_' + suffix + '_link'}"/>
-            <xacro:insert_block name="origin"/>
-            <xacro:insert_block name="axis"/>
-            <xacro:insert_block name="limit"/>
-        </joint>
-        <xacro:if value="${child == ''}">
-            <link name="${bodypart}_${suffix}_link">
-            </link>
-        </xacro:if>
-    </xacro:macro>
-    <xacro:shoulder_template bodypart="shoulder" suffix="yaw" parent="torso">
+    <xacro:bodypart_template bodypart="shoulder" suffix="yaw" parent="torso">
         <origin xyz="0.5 0 0.5"/>
         <axis xyz="0 -1 0" />
         <limit effort="1000" lower="-1.1" upper="1.9" velocity="0.5" />
-    </xacro:shoulder_template>
-    <xacro:shoulder_template bodypart="shoulder" suffix="pitch" parent="yaw">
+    </xacro:bodypart_template>
+    <xacro:bodypart_template bodypart="shoulder" suffix="pitch" parent="yaw">
         <origin xyz="0 0 0"/>
         <axis xyz="0 0 1"/>
         <limit effort="1000" lower="-0.4" upper="3.3" velocity="0.5" />
-    </xacro:shoulder_template>
-    <xacro:shoulder_template bodypart="shoulder" suffix="roll" parent="pitch" child="upperarm">
+    </xacro:bodypart_template>
+    <xacro:bodypart_template bodypart="shoulder" suffix="roll" parent="pitch" child="upperarm">
         <origin xyz="0 0 0"/>
         <axis xyz="1 0 0"/>
         <!-- Bullshit limit for now  -->
         <limit effort="1000" lower="-0.4" upper="3.3" velocity="0.5" />
-    </xacro:shoulder_template>
+    </xacro:bodypart_template>
     <link name="upperarm">
         <visual>
@@ -52,11 +36,15 @@
     </link>
     <!-- ____________________ Elbow joint ___________ -->
-    <joint name="elbow_joint" type="revolute">
-        <parent link="upperarm"/>
-        <child link="forearm"/>
+    <xacro:bodypart_template bodypart="elbow" suffix="yaw" parent="upperarm">
+        <origin xyz="${upperarm_length} 0 0"/>
         <axis xyz="0 0 1" />
         <limit effort="1000" lower="0" upper="2.5" velocity="0.5" />
-        <origin xyz="${upperarm_length} 0 0"/>
-    </joint>
+    </xacro:bodypart_template>
+    <xacro:bodypart_template bodypart="elbow" suffix="roll" parent="yaw" child="forearm">
+        <origin xyz="0 0 0"/>
+        <axis xyz="1 0 0" />
+        <!-- Bullshit limit for now  -->
+        <limit effort="1000" lower="-0.4" upper="3.3" velocity="0.5" />
+    </xacro:bodypart_template>
     <link name="forearm">
         <visual>
@@ -67,3 +55,32 @@
         </visual>
     </link>
+    <!-- ___________________ wrist joint __________ -->
+    <xacro:bodypart_template bodypart="wrist" suffix="yaw" parent="forearm" child="hand">
+        <origin xyz="${elbow_wrist_length} 0 0"/>
+        <axis xyz="0 0 1" />
+        <!-- Bullshit limit for now  -->
+        <limit effort="1000" lower="${(math.pi/180)*45}" upper="${(math.pi/180)*-90}" velocity="0.5" />
+    </xacro:bodypart_template>
+    <link name="hand">
+        <visual>
+            <geometry>
+                <!-- Bullshit limit for now  -->
+                <box size="0.1 0.1 0.1"/>
+            </geometry>
+        </visual>
+    </link>
+    <joint name="hand_can_joint" type="fixed">
+        <parent link="hand"/>
+        <child link="can"/>
+        <!-- Bullshit limit for now  -->
+        <origin xyz="0.05 0.1 0"/>
+    </joint>
+    <link name="can">
+        <visual>
+            <geometry>
+                <!-- Bullshit limit for now  -->
+                <cylinder length="${can_height}" radius="${can_radius}"/>
+            </geometry>
+        </visual>
+    </link>
 </robot>
