Commit message: introduced more constants & approaching realistic model. Still to fix: hand yaw

File: ros2_ws/src/human_arm_model/urdf/constants.urdf.xacro (robot description, xacro)
@@ -1,4 +1,5 @@
 <?xml version="1.0"?>
 <robot xmlns:xacro="http://www.ros.org/wiki/xacro">
+    <!-- Längen -->
     <xacro:property name="upperarm_length" value="0.3637"/>
     <xacro:property name="elbow_wrist_length" value="0.2869"/>
@@ -8,7 +9,19 @@
     <xacro:property name="can_radius" value="0.035"/>
     <xacro:property name="can_height" value="0.12" />
-    <xacro:property name="hand_lenght" value="" />
-    <xacro:property name="hand_height" value="" />
-    <xacro:property name="hand_width" value="" />
+    <xacro:property name="hand_circumference" value="0.2123"/>
+    <!-- Length of handpalm which might be approx. center of can: -->
+    <xacro:property name="hand_lenght" value="0.1165" />
+    <xacro:property name="hand_thickness" value="${(hand_circumference-2*hand_width)/2}" />
+    <xacro:property name="hand_width" value="0.0883" />
+    <!-- Winkel -->
+     <!-- Diese sind Bewegungsamplituden und nicht 1:1 im Model vorwendbar. -->
+    <xacro:property name="shoulder_ab_min" value="${-10*math.pi/180}" />
+    <xacro:property name="shoulder_ab_max" value="${170*math.pi/180}" />
+    <xacro:property name="shoulder_flex_min" value="${-60*math.pi/180}" />
+    <xacro:property name="shoulder_flex_max" value="${170*math.pi/180}" />
+    <xacro:property name="shoulder_rot_min" value="${-60*math.pi/180}" />
+    <xacro:property name="shoulder_rot_max" value="${90*math.pi/180}" />
+    <xacro:property name="elbow_flex_min" value="${-90*math.pi/180}" />
+    <xacro:property name="elbow_flex_max" value="${60*math.pi/180}" />
     <!-- ___________________ Macro for joints __________ -->
     <xacro:macro name="bodypart_template" params="bodypart suffix parent child:='' *origin *axis *limit">

File: ros2_ws/src/human_arm_model/urdf/model.urdf.xacro (robot description, xacro)
@@ -15,4 +15,5 @@
         <axis xyz="0 -1 0" />
         <limit effort="1000" lower="-1.1" upper="1.9" velocity="0.5" />
+        <!-- <limit effort="1000" lower="${shoulder_ab_min}" upper="${shoulder_ab_max}" velocity="0.5" /> -->
     </xacro:bodypart_template>
     <xacro:bodypart_template bodypart="shoulder" suffix="pitch" parent="yaw">
@@ -20,4 +21,5 @@
         <axis xyz="0 0 1"/>
         <limit effort="1000" lower="-0.4" upper="3.3" velocity="0.5" />
+        <!-- <limit effort="1000" lower="${shoulder_flex_min}" upper="${shoulder_flex_max}" velocity="0.5" /> -->
     </xacro:bodypart_template>
     <xacro:bodypart_template bodypart="shoulder" suffix="roll" parent="pitch" child="upperarm">
@@ -25,5 +27,6 @@
         <axis xyz="1 0 0"/>
         <!-- Bullshit limit for now  -->
-        <limit effort="1000" lower="-0.4" upper="3.3" velocity="0.5" />
+        <!-- <limit effort="1000" lower="-0.4" upper="3.3" velocity="0.5" /> -->
+        <limit effort="1000" lower="${shoulder_rot_min}" upper="${shoulder_rot_max}" velocity="0.5" />
     </xacro:bodypart_template>
     <link name="upperarm">
@@ -45,5 +48,5 @@
         <axis xyz="1 0 0" />
         <!-- Bullshit limit for now  -->
-        <limit effort="1000" lower="-0.4" upper="3.3" velocity="0.5" />
+        <limit effort="1000" lower="${(-math.pi/180)*45}" upper="${(math.pi/180)*0}" velocity="0.5" />
     </xacro:bodypart_template>
     <link name="forearm">
@@ -60,12 +63,13 @@
         <axis xyz="0 0 1" />
         <!-- Bullshit limit for now  -->
-        <limit effort="1000" lower="${(math.pi/180)*45}" upper="${(math.pi/180)*-90}" velocity="0.5" />
+        <!-- <limit effort="1000" lower="${(math.pi/180)*45}" upper="${(math.pi/180)*-90}" velocity="0.5" /> -->
+         <limit effort="1000" lower="${(math.pi/180)*45}" upper="${(math.pi/180)*-90}" velocity="0.5" />
     </xacro:bodypart_template>
     <link name="hand">
         <visual>
             <geometry>
-                <!-- Bullshit limit for now  -->
-                <box size="0.1 0.1 0.1"/>
+                <box size="${hand_thickness} ${hand_lenght} ${hand_width}"/>
             </geometry>
+            <origin xyz="${hand_thickness/2} ${hand_lenght/2} 0" rpy="0 0 0"/>
         </visual>
     </link>
@@ -73,13 +77,12 @@
         <parent link="hand"/>
         <child link="can"/>
-        <!-- Bullshit limit for now  -->
-        <origin xyz="0.05 0.1 0"/>
+        <origin xyz="${-hand_thickness/2 } ${hand_lenght} 0"/>
     </joint>
     <link name="can">
         <visual>
             <geometry>
-                <!-- Bullshit limit for now  -->
                 <cylinder length="${can_height}" radius="${can_radius}"/>
             </geometry>
+            <origin xyz="${-can_radius+hand_thickness/2} 0 0"/>
         </visual>
     </link>

Commit message: process of making the model more realistic

File: ros2_ws/src/human_arm_model/urdf/constants.urdf.xacro (robot description, xacro)
@@ -1,5 +1,5 @@
 <?xml version="1.0"?>
 <robot xmlns:xacro="http://www.ros.org/wiki/xacro">
-    <!-- Längen -->
+    <!-- sizes -->
     <xacro:property name="upperarm_length" value="0.3637"/>
     <xacro:property name="elbow_wrist_length" value="0.2869"/>
@@ -11,5 +11,5 @@
     <xacro:property name="hand_circumference" value="0.2123"/>
     <!-- Length of handpalm which might be approx. center of can: -->
-    <xacro:property name="hand_lenght" value="0.1165" />
+    <xacro:property name="hand_length" value="0.1165" />
     <xacro:property name="hand_thickness" value="${(hand_circumference-2*hand_width)/2}" />
     <xacro:property name="hand_width" value="0.0883" />
@@ -24,4 +24,7 @@
     <xacro:property name="elbow_flex_min" value="${-90*math.pi/180}" />
     <xacro:property name="elbow_flex_max" value="${60*math.pi/180}" />
+    <!-- angles from anatomy book -->
+     <xacro:property name="hand_palmarflexion" value="${-85*math.pi /180}" />
+     <xacro:property name="hand_dorsalextension" value="${85*math.pi /180}" />
     <!-- ___________________ Macro for joints __________ -->
     <xacro:macro name="bodypart_template" params="bodypart suffix parent child:='' *origin *axis *limit">

File: ros2_ws/src/human_arm_model/urdf/model.urdf.xacro (robot description, xacro)
@@ -15,5 +15,5 @@
         <axis xyz="0 -1 0" />
         <limit effort="1000" lower="-1.1" upper="1.9" velocity="0.5" />
-        <!-- <limit effort="1000" lower="${shoulder_ab_min}" upper="${shoulder_ab_max}" velocity="0.5" /> -->
+        <!-- <limit effort="1000" lower="${shoulder_flex_max}" upper="${shoulder_flex_min}" velocity="0.5" /> -->
     </xacro:bodypart_template>
     <xacro:bodypart_template bodypart="shoulder" suffix="pitch" parent="yaw">
@@ -21,5 +21,5 @@
         <axis xyz="0 0 1"/>
         <limit effort="1000" lower="-0.4" upper="3.3" velocity="0.5" />
-        <!-- <limit effort="1000" lower="${shoulder_flex_min}" upper="${shoulder_flex_max}" velocity="0.5" /> -->
+        <!-- <limit effort="1000" lower="${shoulder_ab_min}" upper="${shoulder_ab_max}" velocity="0.5" /> -->
     </xacro:bodypart_template>
     <xacro:bodypart_template bodypart="shoulder" suffix="roll" parent="pitch" child="upperarm">
@@ -27,5 +27,5 @@
         <axis xyz="1 0 0"/>
         <!-- Bullshit limit for now  -->
-        <!-- <limit effort="1000" lower="-0.4" upper="3.3" velocity="0.5" /> -->
+        <!-- <limit effort="1000" lower="${60*math.pi/180}" upper="${100*math.pi/180}" velocity="0.5" /> -->
         <limit effort="1000" lower="${shoulder_rot_min}" upper="${shoulder_rot_max}" velocity="0.5" />
     </xacro:bodypart_template>
@@ -64,12 +64,12 @@
         <!-- Bullshit limit for now  -->
         <!-- <limit effort="1000" lower="${(math.pi/180)*45}" upper="${(math.pi/180)*-90}" velocity="0.5" /> -->
-         <limit effort="1000" lower="${(math.pi/180)*45}" upper="${(math.pi/180)*-90}" velocity="0.5" />
+         <limit effort="1000" lower="${hand_palmarflexion}" upper="${hand_dorsalextension}" velocity="0.5" />
     </xacro:bodypart_template>
     <link name="hand">
         <visual>
             <geometry>
-                <box size="${hand_thickness} ${hand_lenght} ${hand_width}"/>
+                <box size="${hand_thickness} ${hand_length} ${hand_width}"/>
             </geometry>
-            <origin xyz="${hand_thickness/2} ${hand_lenght/2} 0" rpy="0 0 0"/>
+            <origin xyz="${hand_length/2} 0 0" rpy="0 0 ${math.pi/2}"/>
         </visual>
     </link>
@@ -77,5 +77,5 @@
         <parent link="hand"/>
         <child link="can"/>
-        <origin xyz="${-hand_thickness/2 } ${hand_lenght} 0"/>
+        <origin xyz="${hand_length} ${hand_thickness/2} 0"/>
     </joint>
     <link name="can">
@@ -84,5 +84,5 @@
                 <cylinder length="${can_height}" radius="${can_radius}"/>
             </geometry>
-            <origin xyz="${-can_radius+hand_thickness/2} 0 0"/>
+            <origin xyz="0 ${can_radius} 0"/>
         </visual>
     </link>

Commit message: exported macros in new file; added new constants. tried implementing alt to model. doesn't work, doesn't launch.

File: ros2_ws/src/human_arm_model/urdf/constants.urdf.xacro (robot description, xacro)
@@ -14,6 +14,10 @@
     <xacro:property name="hand_thickness" value="${(hand_circumference-2*hand_width)/2}" />
     <xacro:property name="hand_width" value="0.0883" />
+    <xacro:property name="waist_back_length" value="0.4776" />
+    <xacro:property name="shoulder_length" value="0.1498" />
+    <xacro:property name="clavicle_link_length" value="0.2081" />
+    <xacro:property name="sternum_radius" value="${clavicle_link_length - shoulder_length}" />
     <!-- Winkel -->
-     <!-- Diese sind Bewegungsamplituden und nicht 1:1 im Model vorwendbar. -->
+    <!-- Diese sind Bewegungsamplituden und nicht 1:1 im Model vorwendbar. -->
     <xacro:property name="shoulder_ab_min" value="${-10*math.pi/180}" />
     <xacro:property name="shoulder_ab_max" value="${170*math.pi/180}" />
@@ -25,19 +29,5 @@
     <xacro:property name="elbow_flex_max" value="${60*math.pi/180}" />
     <!-- angles from anatomy book -->
-     <xacro:property name="hand_palmarflexion" value="${-85*math.pi /180}" />
-     <xacro:property name="hand_dorsalextension" value="${85*math.pi /180}" />
-    <!-- ___________________ Macro for joints __________ -->
-    <xacro:macro name="bodypart_template" params="bodypart suffix parent child:='' *origin *axis *limit">
-        <joint name="${bodypart}_${suffix}_joint" type="revolute">
-            <parent link="${parent if (parent in ['torso', 'upperarm', 'forearm']) else bodypart+'_'+parent+'_link'}"/>
-            <child link="${child if child != '' else bodypart+'_' + suffix + '_link'}"/>
-            <xacro:insert_block name="origin"/>
-            <xacro:insert_block name="axis"/>
-            <xacro:insert_block name="limit"/>
-        </joint>
-        <xacro:if value="${child == ''}">
-            <link name="${bodypart}_${suffix}_link">
-            </link>
-        </xacro:if>
-    </xacro:macro>
+    <xacro:property name="hand_palmarflexion" value="${-85*math.pi /180}" />
+    <xacro:property name="hand_dorsalextension" value="${85*math.pi /180}" />
 </robot>

File: ros2_ws/src/human_arm_model/urdf/model.urdf.xacro (robot description, xacro)
@@ -1,5 +1,6 @@
 <?xml version="1.0"?>
-<robot xmlns:xacro="http://www.ros.org/wiki/xacro" name="human_arm_modell">
+<robot xmlns:xacro="http://www.ros.org/wiki/xacro" name="human_arm_model">
     <xacro:include filename="constants.urdf.xacro" />
+    <xacro:include filename="macros.urdf.xacro" />
     <link name="torso">
         <visual>
