Commit message: adjusted angles of clavicula to be more accurate thus allowing a more realistic movement

File: ros2_ws/src/human_arm_model/urdf/glenohumeral_joint.urdf.xacro (robot description, xacro)
@@ -4,5 +4,5 @@
     <xacro:include filename="macros.urdf.xacro" />
     <xacro:joint_template bodypart="glenohumeral" suffix="yaw" parent="clavicular" child="humerus_yaw" >
-        <origin xyz="0 ${clavicle_link_length} 0" />
+        <origin xyz="0 ${clavicle_link_length} 0" rpy="0 0 ${-30*math.pi/180}"/>
         <axis xyz="1 0 0" />
         <limit effort="1000" lower="${glenohumeraljoint_adduktion}" upper="${glenohumeraljoint_abduktion}" velocity="0.5" />

File: ros2_ws/src/human_arm_model/urdf/sternoclavicular_joint.urdf.xacro (robot description, xacro)
@@ -4,5 +4,5 @@
     <xacro:include filename="macros.urdf.xacro" />
     <xacro:joint_template bodypart="sternoclavicular" suffix="yaw" parent="columna" child="clavicular_yaw" >
-        <origin xyz="0 ${sternum_radius} ${waist_back_length}" />
+        <origin xyz="0 ${sternum_radius} ${waist_back_length}" rpy="0 0 ${30*math.pi/180}" />
         <axis xyz="1 0 0" />
         <limit effort="1000" lower="${Sternoklavikularjoint_depression}" upper="${Sternoklavikularjoint_elevation}" velocity="0.5" />
