Commit message: edited files to hopefully be able to launch gazebo later. Next milestone: building the launch file(s)

File: ros2_ws/src/human_arm_model/urdf/alt_gazebo.urdf.xacro (robot description, xacro)
@@ -2,7 +2,24 @@
 <robot xmlns:xacro="http://www.ros.org/wiki/xacro" name="alt_human_arm_model">
     <xacro:include filename="macros.urdf.xacro" />
+    <!-- <gazebo>
+        <plugin
+            name="gz_ros2_control"
+            filename="gz_ros2_control-system">
+            <ros2_control>
+                <param>/config/config.yaml</param>
+            </ros2_control>
+        </plugin>
+    </gazebo> -->
+    <gazebo>
+        <plugin filename="gz_ros2_control-system" name="gz_ros2_control::GazeboSimROS2ControlPlugin">
+            <parameters>src/human_arm_model/config/config.yaml</parameters>
+            <ros>
+                <remapping>/controller_manager/robot_description:=/robot_description</remapping>
+            </ros>
+        </plugin>
+    </gazebo>
     <ros2_control name="SimHardware" type="system">
         <hardware>
-            <plugin>gazebo_ros2_control/GazeboSystem</plugin>
+            <plugin>gz_ros2_control/GazeboSimSystem</plugin>
         </hardware>
         <xacro:joint_interfaces joint_name="sternoclavicular_yaw_joint"/>
@@ -16,5 +33,5 @@
         <xacro:joint_interfaces joint_name="wrist_yaw_joint"/>
     </ros2_control>
-    <xacro:joint_transmission joint_name="sternoclavicular_yaw_joint" />
+    <!-- <xacro:joint_transmission joint_name="sternoclavicular_yaw_joint" />
     <xacro:joint_transmission joint_name="sternoclavicular_pitch_joint" />
     <xacro:joint_transmission joint_name="sternoclavicular_roll_joint" />
@@ -24,4 +41,4 @@
     <xacro:joint_transmission joint_name="elbow_roll_joint" />
     <xacro:joint_transmission joint_name="elbow_yaw_joint" />
-    <xacro:joint_transmission joint_name="wrist_yaw_joint" />
+    <xacro:joint_transmission joint_name="wrist_yaw_joint" /> -->
 </robot>

File: ros2_ws/src/human_arm_model/urdf/macros.urdf.xacro (robot description, xacro)
@@ -55,10 +55,10 @@
     <xacro:macro name="joint_interfaces" params="joint_name">
         <joint name="${joint_name}">
-            <command_interface name="position"/>
+            <command_interface name="position">
+            </command_interface>
             <state_interface name="position"/>
-            <state_interface name="velocity"/>
         </joint>
     </xacro:macro>
-    <xacro:macro name="joint_transmission" params="joint_name">
+    <!-- <xacro:macro name="joint_transmission" params="joint_name">
         <transmission name="${joint_name}_trans">
         <type>transmission_interface/SimpleTransmission</type>
@@ -71,5 +71,5 @@
         </actuator>
         </transmission>
-    </xacro:macro>
+    </xacro:macro> -->
     <xacro:macro name="minimal_interia">
         <inertial>
