Commit message: alt is now launching, but not displaying yet.

File: ros2_ws/src/human_arm_model/urdf/alt_model.urdf.xacro (robot description, xacro)
@@ -1,4 +1,4 @@
 <?xml version="1.0"?>
-<robot xmlns:xacro="http://www.ros.org/wiki/xacro" name="human_arm_model">
+<robot xmlns:xacro="http://www.ros.org/wiki/xacro" name="alt_human_arm_model">
     <xacro:include filename="constants.urdf.xacro" />
     <xacro:include filename="macros.urdf.xacro" />
@@ -14,12 +14,19 @@
             <!-- 9. hand -->
         <!-- 7. and 8. are simplified significantly, both reduced from 2 subparts to 1, as the complexity is not needed here  -->
+    <link name="world"/>
+    <joint name="world_to_columna" type="fixed">
+        <parent link="world"/>
+        <child link="columna"/>
+        <origin xyz="0 0 0"/>
+    </joint>
     <link name="columna"> <!-- carla columna-->
         <visual>
             <geometry>
                 <box size="${sternum_radius*2} ${sternum_radius*2} ${waist_back_length}"/>
+                <box size="1 1 1"/>
             </geometry>
         </visual>
     </link>
-    <xacro:bodypart_template bodypart="sternoclavicular" suffix="yaw" parent="columna" child="clavicular" >
+    <!-- <xacro:bodypart_template bodypart="sternoclavicular" suffix="yaw" parent="columna" child="clavicular" >
         <origin xyz="0 ${sternum_radius} ${waist_back_length}" />
         <axis xyz="0 -1 0" />
@@ -32,4 +39,4 @@
             </geometry>
         </visual>
-    </link>
+    </link> -->
 </robot>

Commit message: launch of new model works. model created until forearm. elevation of upperarm is still faulty. sternoclavicular joint might not be implemented right

File: ros2_ws/src/human_arm_model/urdf/alt_model.urdf.xacro (robot description, xacro)
@@ -3,4 +3,7 @@
     <xacro:include filename="constants.urdf.xacro" />
     <xacro:include filename="macros.urdf.xacro" />
+    <xacro:include filename="sternoclavicular_joint.urdf.xacro" />
+    <xacro:include filename="glenohumeral_joint.urdf.xacro" />
+    <xacro:include filename="humeroulnar_joint.urdf.xacro" />
     <!-- layout: -->
             <!-- 1. sternum -->
@@ -14,7 +17,7 @@
             <!-- 9. hand -->
         <!-- 7. and 8. are simplified significantly, both reduced from 2 subparts to 1, as the complexity is not needed here  -->
-    <link name="world"/>
+    <link name="base_link"/>
     <joint name="world_to_columna" type="fixed">
-        <parent link="world"/>
+        <parent link="base_link"/>
         <child link="columna"/>
         <origin xyz="0 0 0"/>
@@ -24,18 +27,56 @@
             <geometry>
                 <box size="${sternum_radius*2} ${sternum_radius*2} ${waist_back_length}"/>
-                <box size="1 1 1"/>
             </geometry>
+            <origin xyz="0 0 ${waist_back_length/2}"/>
         </visual>
     </link>
-    <!-- <xacro:bodypart_template bodypart="sternoclavicular" suffix="yaw" parent="columna" child="clavicular" >
-        <origin xyz="0 ${sternum_radius} ${waist_back_length}" />
-        <axis xyz="0 -1 0" />
-        <limit effort="1000" lower="-1.1" upper="1.9" velocity="0.5" />
-    </xacro:bodypart_template>
     <link name="clavicular">
         <visual>
             <geometry>
-                <box size="${sternum_radius*2} ${sternum_radius*2} ${waist_back_length}"/>
+                <cylinder length="${clavicle_link_length}" radius="${sternum_radius/2}"/>
             </geometry>
+            <origin xyz="0 ${clavicle_link_length/2} 0" rpy="${math.pi/2} 0 0"/>
+        </visual>
+    </link>
+    <link name="humerus">
+        <visual>
+            <geometry>
+                <cylinder length="${upperarm_length}" radius="${upperarm_radius}"/>
+            </geometry>
+            <origin xyz="0 0 ${-upperarm_length/2}" rpy="0 0 0"/>
+        </visual>
+    </link>
+    <link name="forearm">
+        <visual>
+            <geometry>
+                <cylinder length="${elbow_wrist_length}" radius="${forearm_circumference / (2*math.pi)}" />
+            </geometry>
+            <origin xyz="0 0 ${-elbow_wrist_length/2}" rpy="0 0 0"/>
+        </visual>
+    </link>
+    <!-- <xacro:bodypart_template bodypart="wrist" suffix="yaw" parent="forearm" child="hand">
+        <origin xyz="${elbow_wrist_length} 0 0"/>
+        <axis xyz="0 0 1" />
+        <limit effort="1000" lower="${hand_palmarflexion}" upper="${hand_dorsalextension}" velocity="0.5" />
+    </xacro:bodypart_template>
+    <link name="hand">
+        <visual>
+            <geometry>
+                <box size="${hand_thickness} ${hand_length} ${hand_width}"/>
+            </geometry>
+            <origin xyz="${hand_length/2} 0 0" rpy="0 0 ${math.pi/2}"/>
+        </visual>
+    </link>
+    <joint name="hand_can_joint" type="fixed">
+        <parent link="hand"/>
+        <child link="can"/>
+        <origin xyz="${hand_length} ${hand_thickness/2} 0"/>
+    </joint>
+    <link name="can">
+        <visual>
+            <geometry>
+                <cylinder length="${can_height}" radius="${can_radius}"/>
+            </geometry>
+            <origin xyz="0 ${can_radius} 0"/>
         </visual>
     </link> -->

File: ros2_ws/src/human_arm_model/urdf/constants.urdf.xacro (robot description, xacro)
@@ -1,4 +1,5 @@
 <?xml version="1.0"?>
 <robot xmlns:xacro="http://www.ros.org/wiki/xacro">
+    <xacro:include filename="macros.urdf.xacro" />
     <!-- sizes -->
     <xacro:property name="upperarm_length" value="0.3637"/>
@@ -28,6 +29,27 @@
     <xacro:property name="elbow_flex_min" value="${-90*math.pi/180}" />
     <xacro:property name="elbow_flex_max" value="${60*math.pi/180}" />
+    <!-- calculated values -->
+    <xacro:property name="upperarm_radius" value="${upperarm_circumference/(2* math.pi)}"/>
     <!-- angles from anatomy book -->
     <xacro:property name="hand_palmarflexion" value="${-85*math.pi /180}" />
     <xacro:property name="hand_dorsalextension" value="${85*math.pi /180}" />
+    <!-- Sternoklavikularjoint -->
+    <xacro:property name="Sternoklavikularjoint_elevation" value="${30*math.pi/180}"/>
+    <xacro:property name="Sternoklavikularjoint_depression" value="${-5*math.pi/180}" />
+    <xacro:property name="Sternoklavikularjoint_protraktion" value="${30*math.pi/180}"/>
+    <xacro:property name="Sternoklavikularjoint_retraktion" value="${-30*math.pi/180}" />
+    <xacro:property name="Sternoklavikularjoint_anteriorrotation" value="${30*math.pi/180}"/>
+    <xacro:property name="Sternoklavikularjoint_posteriorrotation" value="${-30*math.pi/180}" />
+    <!-- Glenohumeraljoint -->
+    <xacro:property name="glenohumeraljoint_abduktion" value="${90*math.pi/180}" />
+    <xacro:property name="glenohumeraljoint_adduktion" value="${0*math.pi/180}" />
+    <xacro:property name="glenohumeraljoint_anteversion" value="${80*math.pi/180}" />
+    <xacro:property name="glenohumeraljoint_retroversion" value="${-40*math.pi/180}" />
+    <xacro:property name="glenohumeraljoint_exorotation" value="${60*math.pi/180}" />
+    <xacro:property name="glenohumeraljoint_endorotation" value="${-100*math.pi/180}" />
+    <!-- Humeroulnarjoint -->
+    <xacro:property name="humeroulnarjoint_flexion" value="${160*math.pi/180}" />
+    <xacro:property name="humeroulnarjoint_extension" value="${-15*math.pi/180}" />
+    <xacro:property name="humeroulnarjoint_pronation" value="${85*math.pi/180}" />
+    <xacro:property name="humeroulnarjoint_supination" value="${-90*math.pi/180}" />
 </robot>

File: ros2_ws/src/human_arm_model/urdf/macros.urdf.xacro (robot description, xacro)
@@ -15,3 +15,12 @@
         </xacro:if>
     </xacro:macro>
+    <xacro:macro name="joint_template" params="bodypart suffix parent child *origin *axis *limit">
+        <joint name="${bodypart}_${suffix}_joint" type="revolute">
+            <parent link="${parent}"/>
+            <child link="${child}" />
+            <xacro:insert_block name="origin"/>
+            <xacro:insert_block name="axis"/>
+            <xacro:insert_block name="limit"/>
+        </joint>
+    </xacro:macro>
 </robot>

Commit message: implemented wrist & can

File: ros2_ws/src/human_arm_model/urdf/alt_model.urdf.xacro (robot description, xacro)
@@ -55,7 +55,7 @@
         </visual>
     </link>
-    <!-- <xacro:bodypart_template bodypart="wrist" suffix="yaw" parent="forearm" child="hand">
-        <origin xyz="${elbow_wrist_length} 0 0"/>
-        <axis xyz="0 0 1" />
+    <xacro:bodypart_template bodypart="wrist" suffix="yaw" parent="forearm" child="hand">
+        <origin xyz="0 0 ${-elbow_wrist_length}"/>
+        <axis xyz="1 0 0" />
         <limit effort="1000" lower="${hand_palmarflexion}" upper="${hand_dorsalextension}" velocity="0.5" />
     </xacro:bodypart_template>
@@ -65,5 +65,5 @@
                 <box size="${hand_thickness} ${hand_length} ${hand_width}"/>
             </geometry>
-            <origin xyz="${hand_length/2} 0 0" rpy="0 0 ${math.pi/2}"/>
+            <origin xyz="0 0 ${-hand_length/2}" rpy="${90*math.pi/180} 0 ${90*math.pi/180}"/>
         </visual>
     </link>
@@ -71,5 +71,5 @@
         <parent link="hand"/>
         <child link="can"/>
-        <origin xyz="${hand_length} ${hand_thickness/2} 0"/>
+        <origin xyz="0 ${-hand_thickness} ${-hand_length} "/>
     </joint>
     <link name="can">
@@ -78,6 +78,6 @@
                 <cylinder length="${can_height}" radius="${can_radius}"/>
             </geometry>
-            <origin xyz="0 ${can_radius} 0"/>
+            <origin xyz="0 0 0" rpy="${90*math.pi/180} 0 ${90*math.pi/180}"/>
         </visual>
-    </link> -->
+    </link>
 </robot>

Commit message: added macro for collision tags and added collision tags in all links

File: ros2_ws/src/human_arm_model/urdf/alt_model.urdf.xacro (robot description, xacro)
@@ -30,29 +30,29 @@
             <origin xyz="0 0 ${waist_back_length/2}"/>
         </visual>
+        <collision>
+            <geometry>
+                <box size="${sternum_radius*2} ${sternum_radius*2} ${waist_back_length}"/>
+            </geometry>
+            <origin xyz="0 0 ${waist_back_length/2}"/>
+        </collision>
     </link>
-    <link name="clavicular">
-        <visual>
-            <geometry>
-                <cylinder length="${clavicle_link_length}" radius="${sternum_radius/2}"/>
-            </geometry>
-            <origin xyz="0 ${clavicle_link_length/2} 0" rpy="${math.pi/2} 0 0"/>
-        </visual>
-    </link>
-    <link name="humerus">
-        <visual>
-            <geometry>
-                <cylinder length="${upperarm_length}" radius="${upperarm_radius}"/>
-            </geometry>
-            <origin xyz="0 0 ${-upperarm_length/2}" rpy="0 0 0"/>
-        </visual>
-    </link>
-    <link name="forearm">
-        <visual>
-            <geometry>
-                <cylinder length="${elbow_wrist_length}" radius="${forearm_circumference / (2*math.pi)}" />
-            </geometry>
-            <origin xyz="0 0 ${-elbow_wrist_length/2}" rpy="0 0 0"/>
-        </visual>
-    </link>
+    <xacro:cylinder_link_template name="clavicular">
+        <geometry>
+            <cylinder length="${clavicle_link_length}" radius="${sternum_radius/2}"/>
+        </geometry>
+        <origin xyz="0 ${clavicle_link_length/2} 0" rpy="${math.pi/2} 0 0"/>
+    </xacro:cylinder_link_template>
+    <xacro:cylinder_link_template name="humerus">
+        <geometry>
+            <cylinder length="${upperarm_length}" radius="${upperarm_radius}"/>
+        </geometry>
+        <origin xyz="0 0 ${-upperarm_length/2}" rpy="0 0 0"/>
+    </xacro:cylinder_link_template>
+    <xacro:cylinder_link_template name="forearm">
+        <geometry>
+            <cylinder length="${elbow_wrist_length}" radius="${forearm_circumference / (2*math.pi)}" />
+        </geometry>
+        <origin xyz="0 0 ${-elbow_wrist_length/2}" rpy="0 0 0"/>
+    </xacro:cylinder_link_template>
     <xacro:bodypart_template bodypart="wrist" suffix="yaw" parent="forearm" child="hand">
         <origin xyz="0 0 ${-elbow_wrist_length}"/>
@@ -67,4 +67,10 @@
             <origin xyz="0 0 ${-hand_length/2}" rpy="${90*math.pi/180} 0 ${90*math.pi/180}"/>
         </visual>
+        <collision>
+            <geometry>
+                <box size="${hand_thickness} ${hand_length} ${hand_width}"/>
+            </geometry>
+            <origin xyz="0 0 ${-hand_length/2}" rpy="${90*math.pi/180} 0 ${90*math.pi/180}"/>
+        </collision>
     </link>
     <joint name="hand_can_joint" type="fixed">
@@ -73,11 +79,9 @@
         <origin xyz="0 ${-hand_thickness} ${-hand_length} "/>
     </joint>
-    <link name="can">
-        <visual>
-            <geometry>
-                <cylinder length="${can_height}" radius="${can_radius}"/>
-            </geometry>
-            <origin xyz="0 0 0" rpy="${90*math.pi/180} 0 ${90*math.pi/180}"/>
-        </visual>
-    </link>
+    <xacro:cylinder_link_template name="can">
+        <geometry>
+            <cylinder length="${can_height}" radius="${can_radius}"/>
+        </geometry>
+        <origin xyz="0 0 0" rpy="${90*math.pi/180} 0 ${90*math.pi/180}"/>
+    </xacro:cylinder_link_template>
 </robot>

File: ros2_ws/src/human_arm_model/urdf/macros.urdf.xacro (robot description, xacro)
@@ -15,4 +15,22 @@
         </xacro:if>
     </xacro:macro>
+    <xacro:macro name="cylinder_link_template"  params="name *origin *geometry">
+        <link name="${name}">
+            <visual>
+                <xacro:insert_block name="origin"/>
+                <xacro:insert_block name="geometry" />
+            </visual>
+            <collision>
+                <xacro:insert_block name="origin"/>
+                <xacro:insert_block name="geometry" />
+            </collision>
+            <!-- <inertial>
+                <xacro:cylinder_inertia>
+                </xacro:cylinder_inertia>
+            </inertial> -->
+        </link>
+    </xacro:macro>
+    <!-- <xacro:macro name="cylinder_inertia">
+    </xacro:macro> -->
     <xacro:macro name="joint_template" params="bodypart suffix parent child *origin *axis *limit">
         <joint name="${bodypart}_${suffix}_joint" type="revolute">

Commit message: changed macro to account for inertia. added inertia to all cylinder links. non cylindric remain. Also mass values set to 1, need to adapt those

File: ros2_ws/src/human_arm_model/urdf/alt_model.urdf.xacro (robot description, xacro)
@@ -37,20 +37,11 @@
         </collision>
     </link>
-    <xacro:cylinder_link_template name="clavicular">
-        <geometry>
-            <cylinder length="${clavicle_link_length}" radius="${sternum_radius/2}"/>
-        </geometry>
+    <xacro:cylinder_link_template name="clavicular" mass="1" radius="${sternum_radius/2}" height="${clavicle_link_length}">
         <origin xyz="0 ${clavicle_link_length/2} 0" rpy="${math.pi/2} 0 0"/>
     </xacro:cylinder_link_template>
-    <xacro:cylinder_link_template name="humerus">
-        <geometry>
-            <cylinder length="${upperarm_length}" radius="${upperarm_radius}"/>
-        </geometry>
+    <xacro:cylinder_link_template name="humerus" mass="1" radius="${upperarm_radius}" height="${upperarm_length}">
         <origin xyz="0 0 ${-upperarm_length/2}" rpy="0 0 0"/>
     </xacro:cylinder_link_template>
-    <xacro:cylinder_link_template name="forearm">
-        <geometry>
-            <cylinder length="${elbow_wrist_length}" radius="${forearm_circumference / (2*math.pi)}" />
-        </geometry>
+    <xacro:cylinder_link_template name="forearm" mass="1" radius="${forearm_circumference / (2*math.pi)}" height="${elbow_wrist_length}">
         <origin xyz="0 0 ${-elbow_wrist_length/2}" rpy="0 0 0"/>
     </xacro:cylinder_link_template>
@@ -79,8 +70,5 @@
         <origin xyz="0 ${-hand_thickness} ${-hand_length} "/>
     </joint>
-    <xacro:cylinder_link_template name="can">
-        <geometry>
-            <cylinder length="${can_height}" radius="${can_radius}"/>
-        </geometry>
+    <xacro:cylinder_link_template name="can" mass="1" radius="${can_radius}" height="${can_height}">
         <origin xyz="0 0 0" rpy="${90*math.pi/180} 0 ${90*math.pi/180}"/>
     </xacro:cylinder_link_template>

File: ros2_ws/src/human_arm_model/urdf/macros.urdf.xacro (robot description, xacro)
@@ -15,22 +15,27 @@
         </xacro:if>
     </xacro:macro>
-    <xacro:macro name="cylinder_link_template"  params="name *origin *geometry">
+    <xacro:macro name="cylinder_link_template"  params="name mass radius height *origin ">
         <link name="${name}">
             <visual>
+                <geometry>
+                    <cylinder length="${height}" radius="${radius}"/>
+                </geometry>
                 <xacro:insert_block name="origin"/>
-                <xacro:insert_block name="geometry" />
             </visual>
             <collision>
                 <xacro:insert_block name="origin"/>
-                <xacro:insert_block name="geometry" />
+                <geometry>
+                    <cylinder length="${height}" radius="${radius}"/>
+                </geometry>
             </collision>
-            <!-- <inertial>
-                <xacro:cylinder_inertia>
-                </xacro:cylinder_inertia>
-            </inertial> -->
+            <xacro:cylinder_inertia m="${mass}" r="${radius}" h="${height}"/>
         </link>
     </xacro:macro>
-    <!-- <xacro:macro name="cylinder_inertia">
-    </xacro:macro> -->
+    <xacro:macro name="cylinder_inertia" params="m r h">
+        <inertial>
+            <mass value="${m}"/>
+            <inertia ixx="${(1/12)* m*(3*r*r + h*h) }" ixy="0.0" ixz="0.0" iyy="${(1/12)* m*(3*r*r + h*h) }" iyz="0.0" izz="${(1/2)*m*r*r}" />
+        </inertial>
+    </xacro:macro>
     <xacro:macro name="joint_template" params="bodypart suffix parent child *origin *axis *limit">
         <joint name="${bodypart}_${suffix}_joint" type="revolute">

Commit message: added mass + inertia for all but columna; clavicula still has mass value 1 as placehiolder

File: ros2_ws/src/human_arm_model/urdf/alt_model.urdf.xacro (robot description, xacro)
@@ -37,11 +37,12 @@
         </collision>
     </link>
+    <!-- placeholder mass here -->
     <xacro:cylinder_link_template name="clavicular" mass="1" radius="${sternum_radius/2}" height="${clavicle_link_length}">
         <origin xyz="0 ${clavicle_link_length/2} 0" rpy="${math.pi/2} 0 0"/>
     </xacro:cylinder_link_template>
-    <xacro:cylinder_link_template name="humerus" mass="1" radius="${upperarm_radius}" height="${upperarm_length}">
+    <xacro:cylinder_link_template name="humerus" mass="${upperarm_weight}" radius="${upperarm_radius}" height="${upperarm_length}">
         <origin xyz="0 0 ${-upperarm_length/2}" rpy="0 0 0"/>
     </xacro:cylinder_link_template>
-    <xacro:cylinder_link_template name="forearm" mass="1" radius="${forearm_circumference / (2*math.pi)}" height="${elbow_wrist_length}">
+    <xacro:cylinder_link_template name="forearm" mass="${forearm_weight}" radius="${forearm_circumference / (2*math.pi)}" height="${elbow_wrist_length}">
         <origin xyz="0 0 ${-elbow_wrist_length/2}" rpy="0 0 0"/>
     </xacro:cylinder_link_template>
@@ -64,4 +65,5 @@
             <origin xyz="0 0 ${-hand_length/2}" rpy="${90*math.pi/180} 0 ${90*math.pi/180}"/>
         </collision>
+        <xacro:box_inertia m="${hand_weight}" x="${hand_thickness}" y="${hand_length}" z="${hand_width}" />
     </link>
     <joint name="hand_can_joint" type="fixed">
@@ -70,5 +72,5 @@
         <origin xyz="0 ${-hand_thickness} ${-hand_length} "/>
     </joint>
-    <xacro:cylinder_link_template name="can" mass="1" radius="${can_radius}" height="${can_height}">
+    <xacro:cylinder_link_template name="can" mass="${can_weight}" radius="${can_radius}" height="${can_height}">
         <origin xyz="0 0 0" rpy="${90*math.pi/180} 0 ${90*math.pi/180}"/>
     </xacro:cylinder_link_template>

File: ros2_ws/src/human_arm_model/urdf/constants.urdf.xacro (robot description, xacro)
@@ -53,3 +53,9 @@
     <xacro:property name="humeroulnarjoint_pronation" value="${85*math.pi/180}" />
     <xacro:property name="humeroulnarjoint_supination" value="${-90*math.pi/180}" />
+    <!-- weights as percentage of whole body -->
+    <xacro:property name="bodyweight" value="85.8"/>
+    <xacro:property name="upperarm_weight" value="${bodyweight * 0.029}"/>
+    <xacro:property name="forearm_weight" value="${bodyweight * 0.017}" />
+    <xacro:property name="hand_weight" value="${bodyweight * 0.007}" />
+    <xacro:property name="can_weight" value="0.45"/>
 </robot>

File: ros2_ws/src/human_arm_model/urdf/macros.urdf.xacro (robot description, xacro)
@@ -38,4 +38,10 @@
         </inertial>
     </xacro:macro>
+    <xacro:macro name="box_inertia" params="m x y z">
+        <inertial>
+            <mass value="${m}"/>
+            <inertia ixx="${(1/12)* m*(y*y + z*z) }" ixy="0.0" ixz="0.0" iyy="${(1/12)* m*(x*x + z*z) }" iyz="0.0" izz="${(1/12)*m* (x*x + y*y)}" />
+        </inertial>
+    </xacro:macro>
     <xacro:macro name="joint_template" params="bodypart suffix parent child *origin *axis *limit">
         <joint name="${bodypart}_${suffix}_joint" type="revolute">

Commit message: added tags for gezebo sim

File: ros2_ws/src/human_arm_model/urdf/alt_model.urdf.xacro (robot description, xacro)
@@ -6,4 +6,5 @@
     <xacro:include filename="glenohumeral_joint.urdf.xacro" />
     <xacro:include filename="humeroulnar_joint.urdf.xacro" />
+    <xacro:include filename="alt_gazebo.urdf.xacro" />
     <!-- layout: -->
             <!-- 1. sternum -->

File: ros2_ws/src/human_arm_model/urdf/macros.urdf.xacro (robot description, xacro)
@@ -53,3 +53,22 @@
         </joint>
     </xacro:macro>
+    <xacro:macro name="joint_interfaces" params="joint_name">
+        <joint name="${joint_name}">
+            <command_interface name="position"/>
+            <state_interface name="position"/>
+            <state_interface name="velocity"/>
+        </joint>
+    </xacro:macro>
+    <xacro:macro name="joint_transmission" params="joint_name">
+        <transmission name="${joint_name}_trans">
+        <type>transmission_interface/SimpleTransmission</type>
+        <joint name="${joint_name}">
+            <hardwareInterface>hardware_interface/PositionCommandInterface</hardwareInterface>
+        </joint>
+        <actuator name="${joint_name}_motor">
+            <hardwareInterface>hardware_interface/PositionCommandInterface</hardwareInterface>
+            <mechanicalReduction>1</mechanicalReduction>
+        </actuator>
+        </transmission>
+    </xacro:macro>
 </robot>
