Commit message: added minimal inertia to all links for Gazebo to work

File: ros2_ws/src/human_arm_model/urdf/alt_model.urdf.xacro (robot description, xacro)
@@ -18,5 +18,7 @@
             <!-- 9. hand -->
         <!-- 7. and 8. are simplified significantly, both reduced from 2 subparts to 1, as the complexity is not needed here  -->
-    <link name="base_link"/>
+    <link name="base_link">
+        <xacro:minimal_interia />
+    </link>
     <joint name="world_to_columna" type="fixed">
         <parent link="base_link"/>
@@ -27,14 +29,15 @@
         <visual>
             <geometry>
-                <box size="${sternum_radius*2} ${sternum_radius*2} ${waist_back_length}"/>
+                <box size="${sternum_radius*2} ${sternum_radius*2} ${2*waist_back_length}"/>
             </geometry>
-            <origin xyz="0 0 ${waist_back_length/2}"/>
+            <origin xyz="0 0 ${waist_back_length}"/>
         </visual>
         <collision>
             <geometry>
-                <box size="${sternum_radius*2} ${sternum_radius*2} ${waist_back_length}"/>
+                <box size="${sternum_radius*2} ${sternum_radius*2} ${2*waist_back_length}"/>
             </geometry>
-            <origin xyz="0 0 ${waist_back_length/2}"/>
+            <origin xyz="0 0 ${waist_back_length}"/>
         </collision>
+        <xacro:box_inertia m="50" x="${sternum_radius*2}" y="${sternum_radius*2}" z="${2*waist_back_length}" />
     </link>
     <!-- placeholder mass here -->

File: ros2_ws/src/human_arm_model/urdf/glenohumeral_joint.urdf.xacro (robot description, xacro)
@@ -8,5 +8,7 @@
         <limit effort="1000" lower="${glenohumeraljoint_adduktion}" upper="${glenohumeraljoint_abduktion}" velocity="0.5" />
     </xacro:joint_template>
-    <link name="humerus_yaw"/>
+    <link name="humerus_yaw">
+        <xacro:minimal_interia />
+    </link>
     <xacro:joint_template bodypart="glenohumeral" suffix="pitch" parent="humerus_yaw" child="humerus_pitch">
         <origin xyz="0 0 0" />
@@ -14,5 +16,7 @@
         <limit effort="1000" lower="${glenohumeraljoint_retroversion}" upper="${glenohumeraljoint_anteversion}" velocity="0.5" />
     </xacro:joint_template>
-    <link name="humerus_pitch"/>
+    <link name="humerus_pitch">
+        <xacro:minimal_interia />
+    </link>
     <xacro:joint_template bodypart="glenohumeral" suffix="roll" parent="humerus_pitch" child="humerus">
         <origin xyz="0 0 0" />

File: ros2_ws/src/human_arm_model/urdf/humeroulnar_joint.urdf.xacro (robot description, xacro)
@@ -8,5 +8,7 @@
         <limit effort="1000" lower="${humeroulnarjoint_extension}" upper="${humeroulnarjoint_flexion}" velocity="0.5" />
     </xacro:joint_template>
-    <link name="forearm_yaw"/>
+    <link name="forearm_yaw">
+        <xacro:minimal_interia />
+    </link>
     <xacro:joint_template bodypart="elbow" suffix="roll" parent="forearm_yaw" child="forearm">
         <origin xyz="0 0 0"/>

File: ros2_ws/src/human_arm_model/urdf/macros.urdf.xacro (robot description, xacro)
@@ -72,3 +72,10 @@
         </transmission>
     </xacro:macro>
+    <xacro:macro name="minimal_interia">
+        <inertial>
+            <origin xyz="0 0 0" rpy="0 0 0"/>
+            <mass value="0.01"/>
+            <inertia ixx="0.001" ixy="0" ixz="0" iyy="0.001" iyz="0" izz="0.001"/>
+        </inertial>
+    </xacro:macro>
 </robot>

File: ros2_ws/src/human_arm_model/urdf/sternoclavicular_joint.urdf.xacro (robot description, xacro)
@@ -4,9 +4,11 @@
     <xacro:include filename="macros.urdf.xacro" />
     <xacro:joint_template bodypart="sternoclavicular" suffix="yaw" parent="columna" child="clavicular_yaw" >
-        <origin xyz="0 ${sternum_radius} ${waist_back_length}" rpy="0 0 ${30*math.pi/180}" />
+        <origin xyz="0 ${sternum_radius} ${2*waist_back_length}" rpy="0 0 ${30*math.pi/180}" />
         <axis xyz="1 0 0" />
         <limit effort="1000" lower="${Sternoklavikularjoint_depression}" upper="${Sternoklavikularjoint_elevation}" velocity="0.5" />
     </xacro:joint_template>
-    <link name="clavicular_yaw"/>
+    <link name="clavicular_yaw">
+        <xacro:minimal_interia />
+    </link>
     <xacro:joint_template bodypart="sternoclavicular" suffix="pitch" parent="clavicular_yaw" child="clavicular_pitch">
         <origin xyz="0 0 0" />
@@ -14,5 +16,7 @@
         <limit effort="1000" lower="${Sternoklavikularjoint_retraktion}" upper="${Sternoklavikularjoint_protraktion}" velocity="0.5" />
     </xacro:joint_template>
-    <link name="clavicular_pitch"/>
+    <link name="clavicular_pitch">
+        <xacro:minimal_interia />
+    </link>
     <xacro:joint_template bodypart="sternoclavicular" suffix="roll" parent="clavicular_pitch" child="clavicular">
         <origin xyz="0 0 0" />

Commit message: changed order of joints and links, to maybe be able to load urdf into MoveIt Wizard

File: ros2_ws/src/human_arm_model/urdf/alt_model.urdf.xacro (robot description, xacro)
@@ -3,8 +3,4 @@
     <xacro:include filename="constants.urdf.xacro" />
     <xacro:include filename="macros.urdf.xacro" />
-    <xacro:include filename="sternoclavicular_joint.urdf.xacro" />
-    <xacro:include filename="glenohumeral_joint.urdf.xacro" />
-    <xacro:include filename="humeroulnar_joint.urdf.xacro" />
-    <xacro:include filename="alt_gazebo.urdf.xacro" />
     <!-- layout: -->
             <!-- 1. sternum -->
@@ -21,9 +17,4 @@
         <!-- <xacro:minimal_interia /> -->
     </link>
-    <joint name="world_to_columna" type="fixed">
-        <parent link="base_link"/>
-        <child link="columna"/>
-        <origin xyz="0 0 0"/>
-    </joint>
     <link name="columna"> <!-- carla columna-->
         <visual>
@@ -41,4 +32,9 @@
         <xacro:box_inertia m="50" x="${sternum_radius*2}" y="${sternum_radius*2}" z="${2*waist_back_length}" />
     </link>
+    <joint name="world_to_columna" type="fixed">
+        <parent link="base_link"/>
+        <child link="columna"/>
+        <origin xyz="0 0 0"/>
+    </joint>
     <!-- placeholder mass here -->
     <xacro:cylinder_link_template name="clavicular" mass="1" radius="${sternum_radius/2}" height="${clavicle_link_length}">
@@ -71,4 +67,7 @@
         <xacro:box_inertia m="${hand_weight}" x="${hand_thickness}" y="${hand_length}" z="${hand_width}" />
     </link>
+    <xacro:cylinder_link_template name="can" mass="${can_weight}" radius="${can_radius}" height="${can_height}">
+        <origin xyz="0 0 0" rpy="${90*math.pi/180} 0 ${90*math.pi/180}"/>
+    </xacro:cylinder_link_template>
     <joint name="hand_can_joint" type="fixed">
         <parent link="hand"/>
@@ -76,6 +75,7 @@
         <origin xyz="0 ${-hand_thickness} ${-hand_length} "/>
     </joint>
-    <xacro:cylinder_link_template name="can" mass="${can_weight}" radius="${can_radius}" height="${can_height}">
-        <origin xyz="0 0 0" rpy="${90*math.pi/180} 0 ${90*math.pi/180}"/>
-    </xacro:cylinder_link_template>
+    <xacro:include filename="sternoclavicular_joint.urdf.xacro" />
+    <xacro:include filename="glenohumeral_joint.urdf.xacro" />
+    <xacro:include filename="humeroulnar_joint.urdf.xacro" />
+    <xacro:include filename="alt_gazebo.urdf.xacro" />
 </robot>

File: ros2_ws/src/human_arm_model/urdf/glenohumeral_joint.urdf.xacro (robot description, xacro)
@@ -3,4 +3,10 @@
     <xacro:include filename="constants.urdf.xacro" />
     <xacro:include filename="macros.urdf.xacro" />
+    <link name="humerus_yaw">
+        <xacro:minimal_interia />
+    </link>
+    <link name="humerus_pitch">
+        <xacro:minimal_interia />
+    </link>
     <xacro:joint_template bodypart="glenohumeral" suffix="yaw" parent="clavicular" child="humerus_yaw" >
         <origin xyz="0 ${clavicle_link_length} 0" rpy="0 0 ${-30*math.pi/180}"/>
@@ -8,7 +14,4 @@
         <limit effort="1000" lower="${glenohumeraljoint_adduktion}" upper="${glenohumeraljoint_abduktion}" velocity="0.5" />
     </xacro:joint_template>
-    <link name="humerus_yaw">
-        <xacro:minimal_interia />
-    </link>
     <xacro:joint_template bodypart="glenohumeral" suffix="pitch" parent="humerus_yaw" child="humerus_pitch">
         <origin xyz="0 0 0" />
@@ -16,7 +19,4 @@
         <limit effort="1000" lower="${glenohumeraljoint_retroversion}" upper="${glenohumeraljoint_anteversion}" velocity="0.5" />
     </xacro:joint_template>
-    <link name="humerus_pitch">
-        <xacro:minimal_interia />
-    </link>
     <xacro:joint_template bodypart="glenohumeral" suffix="roll" parent="humerus_pitch" child="humerus">
         <origin xyz="0 0 0" />

File: ros2_ws/src/human_arm_model/urdf/humeroulnar_joint.urdf.xacro (robot description, xacro)
@@ -3,4 +3,7 @@
     <xacro:include filename="constants.urdf.xacro" />
     <xacro:include filename="macros.urdf.xacro" />
+    <link name="forearm_yaw">
+        <xacro:minimal_interia />
+    </link>
     <xacro:joint_template bodypart="elbow" suffix="yaw" parent="humerus" child="forearm_yaw">
         <origin xyz="0 0 ${-upperarm_length}"/>
@@ -8,7 +11,4 @@
         <limit effort="1000" lower="${humeroulnarjoint_extension}" upper="${humeroulnarjoint_flexion}" velocity="0.5" />
     </xacro:joint_template>
-    <link name="forearm_yaw">
-        <xacro:minimal_interia />
-    </link>
     <xacro:joint_template bodypart="elbow" suffix="roll" parent="forearm_yaw" child="forearm">
         <origin xyz="0 0 0"/>

File: ros2_ws/src/human_arm_model/urdf/macros.urdf.xacro (robot description, xacro)
@@ -3,4 +3,8 @@
     <!-- ___________________ Macro for joints __________ -->
     <xacro:macro name="bodypart_template" params="bodypart suffix parent child:='' *origin *axis *limit">
+        <xacro:if value="${child == ''}">
+            <link name="${bodypart}_${suffix}_link">
+            </link>
+        </xacro:if>
         <joint name="${bodypart}_${suffix}_joint" type="revolute">
             <parent link="${parent if (parent in ['torso', 'upperarm', 'forearm']) else bodypart+'_'+parent+'_link'}"/>
@@ -10,8 +14,4 @@
             <xacro:insert_block name="limit"/>
         </joint>
-        <xacro:if value="${child == ''}">
-            <link name="${bodypart}_${suffix}_link">
-            </link>
-        </xacro:if>
     </xacro:macro>
     <xacro:macro name="cylinder_link_template"  params="name mass radius height *origin ">

File: ros2_ws/src/human_arm_model/urdf/sternoclavicular_joint.urdf.xacro (robot description, xacro)
@@ -3,4 +3,10 @@
     <xacro:include filename="constants.urdf.xacro" />
     <xacro:include filename="macros.urdf.xacro" />
+    <link name="clavicular_yaw">
+        <xacro:minimal_interia />
+    </link>
+    <link name="clavicular_pitch">
+        <xacro:minimal_interia />
+    </link>
     <xacro:joint_template bodypart="sternoclavicular" suffix="yaw" parent="columna" child="clavicular_yaw" >
         <origin xyz="0 ${sternum_radius} ${2*waist_back_length}" rpy="0 0 ${30*math.pi/180}" />
@@ -8,7 +14,4 @@
         <limit effort="1000" lower="${Sternoklavikularjoint_depression}" upper="${Sternoklavikularjoint_elevation}" velocity="0.5" />
     </xacro:joint_template>
-    <link name="clavicular_yaw">
-        <xacro:minimal_interia />
-    </link>
     <xacro:joint_template bodypart="sternoclavicular" suffix="pitch" parent="clavicular_yaw" child="clavicular_pitch">
         <origin xyz="0 0 0" />
@@ -16,7 +19,4 @@
         <limit effort="1000" lower="${Sternoklavikularjoint_retraktion}" upper="${Sternoklavikularjoint_protraktion}" velocity="0.5" />
     </xacro:joint_template>
-    <link name="clavicular_pitch">
-        <xacro:minimal_interia />
-    </link>
     <xacro:joint_template bodypart="sternoclavicular" suffix="roll" parent="clavicular_pitch" child="clavicular">
         <origin xyz="0 0 0" />

Commit message: added .0 to every integer-like number

File: ros2_ws/src/human_arm_model/urdf/alt_model.urdf.xacro (robot description, xacro)
@@ -22,5 +22,5 @@
                 <box size="${sternum_radius*2} ${sternum_radius*2} ${2*waist_back_length}"/>
             </geometry>
-            <origin xyz="0 0 ${waist_back_length}"/>
+            <origin xyz="0.0 0.0 ${waist_back_length}"/>
         </visual>
         <collision>
@@ -28,27 +28,27 @@
                 <box size="${sternum_radius*2} ${sternum_radius*2} ${2*waist_back_length}"/>
             </geometry>
-            <origin xyz="0 0 ${waist_back_length}"/>
+            <origin xyz="0.0 0.0 ${waist_back_length}"/>
         </collision>
-        <xacro:box_inertia m="50" x="${sternum_radius*2}" y="${sternum_radius*2}" z="${2*waist_back_length}" />
+        <xacro:box_inertia m="50.0" x="${sternum_radius*2}" y="${sternum_radius*2}" z="${2*waist_back_length}" />
     </link>
     <joint name="world_to_columna" type="fixed">
         <parent link="base_link"/>
         <child link="columna"/>
-        <origin xyz="0 0 0"/>
+        <origin xyz="0.0 0.0 0.0"/>
     </joint>
     <!-- placeholder mass here -->
     <xacro:cylinder_link_template name="clavicular" mass="1" radius="${sternum_radius/2}" height="${clavicle_link_length}">
-        <origin xyz="0 ${clavicle_link_length/2} 0" rpy="${math.pi/2} 0 0"/>
+        <origin xyz="0.0 ${clavicle_link_length/2} 0.0" rpy="${math.pi/2} 0.0 0.0"/>
     </xacro:cylinder_link_template>
     <xacro:cylinder_link_template name="humerus" mass="${upperarm_weight}" radius="${upperarm_radius}" height="${upperarm_length}">
-        <origin xyz="0 0 ${-upperarm_length/2}" rpy="0 0 0"/>
+        <origin xyz="0.0 0.0 ${-upperarm_length/2}" rpy="0.0 0.0 0.0"/>
     </xacro:cylinder_link_template>
     <xacro:cylinder_link_template name="forearm" mass="${forearm_weight}" radius="${forearm_circumference / (2*math.pi)}" height="${elbow_wrist_length}">
-        <origin xyz="0 0 ${-elbow_wrist_length/2}" rpy="0 0 0"/>
+        <origin xyz="0.0 0.0 ${-elbow_wrist_length/2}" rpy="0.0 0.0 0.0"/>
     </xacro:cylinder_link_template>
     <xacro:bodypart_template bodypart="wrist" suffix="yaw" parent="forearm" child="hand">
-        <origin xyz="0 0 ${-elbow_wrist_length}"/>
-        <axis xyz="1 0 0" />
-        <limit effort="1000" lower="${hand_palmarflexion}" upper="${hand_dorsalextension}" velocity="0.5" />
+        <origin xyz="0.0 0.0 ${-elbow_wrist_length}"/>
+        <axis xyz="1.0 0.0 0.0" />
+        <limit effort="1000.0" lower="${hand_palmarflexion}" upper="${hand_dorsalextension}" velocity="0.5" />
     </xacro:bodypart_template>
     <link name="hand">
@@ -57,5 +57,5 @@
                 <box size="${hand_thickness} ${hand_length} ${hand_width}"/>
             </geometry>
-            <origin xyz="0 0 ${-hand_length/2}" rpy="${90*math.pi/180} 0 ${90*math.pi/180}"/>
+            <origin xyz="0.0 0.0 ${-hand_length/2}" rpy="${90*math.pi/180} 0.0 ${90*math.pi/180}"/>
         </visual>
         <collision>
@@ -63,15 +63,15 @@
                 <box size="${hand_thickness} ${hand_length} ${hand_width}"/>
             </geometry>
-            <origin xyz="0 0 ${-hand_length/2}" rpy="${90*math.pi/180} 0 ${90*math.pi/180}"/>
+            <origin xyz="0.0 0.0 ${-hand_length/2}" rpy="${90*math.pi/180} 0.0 ${90*math.pi/180}"/>
         </collision>
         <xacro:box_inertia m="${hand_weight}" x="${hand_thickness}" y="${hand_length}" z="${hand_width}" />
     </link>
     <xacro:cylinder_link_template name="can" mass="${can_weight}" radius="${can_radius}" height="${can_height}">
-        <origin xyz="0 0 0" rpy="${90*math.pi/180} 0 ${90*math.pi/180}"/>
+        <origin xyz="0.0 0.0 0.0" rpy="${90*math.pi/180} 0.0 ${90*math.pi/180}"/>
     </xacro:cylinder_link_template>
     <joint name="hand_can_joint" type="fixed">
         <parent link="hand"/>
         <child link="can"/>
-        <origin xyz="0 ${-hand_thickness} ${-hand_length} "/>
+        <origin xyz="0.0 ${-hand_thickness} ${-hand_length} "/>
     </joint>
     <xacro:include filename="sternoclavicular_joint.urdf.xacro" />

File: ros2_ws/src/human_arm_model/urdf/glenohumeral_joint.urdf.xacro (robot description, xacro)
@@ -10,17 +10,17 @@
     </link>
     <xacro:joint_template bodypart="glenohumeral" suffix="yaw" parent="clavicular" child="humerus_yaw" >
-        <origin xyz="0 ${clavicle_link_length} 0" rpy="0 0 ${-30*math.pi/180}"/>
-        <axis xyz="1 0 0" />
-        <limit effort="1000" lower="${glenohumeraljoint_adduktion}" upper="${glenohumeraljoint_abduktion}" velocity="0.5" />
+        <origin xyz="0.0 ${clavicle_link_length} 0.0" rpy="0.0 0.0 ${-30*math.pi/180}"/>
+        <axis xyz="1.0 0.0 0.0" />
+        <limit effort="1000.0" lower="${glenohumeraljoint_adduktion}" upper="${glenohumeraljoint_abduktion}" velocity="0.5" />
     </xacro:joint_template>
     <xacro:joint_template bodypart="glenohumeral" suffix="pitch" parent="humerus_yaw" child="humerus_pitch">
-        <origin xyz="0 0 0" />
-        <axis xyz="0 -1 0" />
-        <limit effort="1000" lower="${glenohumeraljoint_retroversion}" upper="${glenohumeraljoint_anteversion}" velocity="0.5" />
+        <origin xyz="0.0 0.0 0.0" />
+        <axis xyz="0.0 -1.0 0.0" />
+        <limit effort="1000.0" lower="${glenohumeraljoint_retroversion}" upper="${glenohumeraljoint_anteversion}" velocity="0.5" />
     </xacro:joint_template>
     <xacro:joint_template bodypart="glenohumeral" suffix="roll" parent="humerus_pitch" child="humerus">
-        <origin xyz="0 0 0" />
-        <axis xyz="0 0 1" />
-        <limit effort="1000" lower="${glenohumeraljoint_endorotation}" upper="${glenohumeraljoint_exorotation}" velocity="0.5" />
+        <origin xyz="0.0 0.0 0.0" />
+        <axis xyz="0.0 0.0 1.0" />
+        <limit effort="1000.0" lower="${glenohumeraljoint_endorotation}" upper="${glenohumeraljoint_exorotation}" velocity="0.5" />
     </xacro:joint_template>
 </robot>

File: ros2_ws/src/human_arm_model/urdf/humeroulnar_joint.urdf.xacro (robot description, xacro)
@@ -7,12 +7,12 @@
     </link>
     <xacro:joint_template bodypart="elbow" suffix="yaw" parent="humerus" child="forearm_yaw">
-        <origin xyz="0 0 ${-upperarm_length}"/>
-        <axis xyz="0 -1 0" />
-        <limit effort="1000" lower="${humeroulnarjoint_extension}" upper="${humeroulnarjoint_flexion}" velocity="0.5" />
+        <origin xyz="0.0 0.0 ${-upperarm_length}"/>
+        <axis xyz="0.0 -1.0 0.0" />
+        <limit effort="1000.0" lower="${humeroulnarjoint_extension}" upper="${humeroulnarjoint_flexion}" velocity="0.5" />
     </xacro:joint_template>
     <xacro:joint_template bodypart="elbow" suffix="roll" parent="forearm_yaw" child="forearm">
-        <origin xyz="0 0 0"/>
-        <axis xyz="0 0 1" />
-        <limit effort="1000" lower="${humeroulnarjoint_supination}" upper="${humeroulnarjoint_pronation}" velocity="0.5" />
+        <origin xyz="0.0 0.0 0.0"/>
+        <axis xyz="0.0 0.0 1.0" />
+        <limit effort="1000.0" lower="${humeroulnarjoint_supination}" upper="${humeroulnarjoint_pronation}" velocity="0.5" />
     </xacro:joint_template>
 </robot>

File: ros2_ws/src/human_arm_model/urdf/macros.urdf.xacro (robot description, xacro)
@@ -74,7 +74,7 @@
     <xacro:macro name="minimal_interia">
         <inertial>
-            <origin xyz="0 0 0" rpy="0 0 0"/>
+            <origin xyz="0.0 0.0 0.0" rpy="0.0 0.0 0.0"/>
             <mass value="0.01"/>
-            <inertia ixx="0.001" ixy="0" ixz="0" iyy="0.001" iyz="0" izz="0.001"/>
+            <inertia ixx="0.001" ixy="0" ixz="0.0" iyy="0.001" iyz="0.0" izz="0.001"/>
         </inertial>
     </xacro:macro>

File: ros2_ws/src/human_arm_model/urdf/sternoclavicular_joint.urdf.xacro (robot description, xacro)
@@ -10,17 +10,17 @@
     </link>
     <xacro:joint_template bodypart="sternoclavicular" suffix="yaw" parent="columna" child="clavicular_yaw" >
-        <origin xyz="0 ${sternum_radius} ${2*waist_back_length}" rpy="0 0 ${30*math.pi/180}" />
-        <axis xyz="1 0 0" />
-        <limit effort="1000" lower="${Sternoklavikularjoint_depression}" upper="${Sternoklavikularjoint_elevation}" velocity="0.5" />
+        <origin xyz="0.0 ${sternum_radius} ${2*waist_back_length}" rpy="0.0 0.0 ${30*math.pi/180}" />
+        <axis xyz="1.0 0.0 0.0" />
+        <limit effort="1000.0" lower="${Sternoklavikularjoint_depression}" upper="${Sternoklavikularjoint_elevation}" velocity="0.5" />
     </xacro:joint_template>
     <xacro:joint_template bodypart="sternoclavicular" suffix="pitch" parent="clavicular_yaw" child="clavicular_pitch">
-        <origin xyz="0 0 0" />
-        <axis xyz="0 0 1" />
-        <limit effort="1000" lower="${Sternoklavikularjoint_retraktion}" upper="${Sternoklavikularjoint_protraktion}" velocity="0.5" />
+        <origin xyz="0.0 0.0 0.0" />
+        <axis xyz="0.0 0.0 1.0" />
+        <limit effort="1000.0" lower="${Sternoklavikularjoint_retraktion}" upper="${Sternoklavikularjoint_protraktion}" velocity="0.5" />
     </xacro:joint_template>
     <xacro:joint_template bodypart="sternoclavicular" suffix="roll" parent="clavicular_pitch" child="clavicular">
-        <origin xyz="0 0 0" />
-        <axis xyz="0 1 0" />
-        <limit effort="1000" lower="${Sternoklavikularjoint_posteriorrotation}" upper="${Sternoklavikularjoint_anteriorrotation}" velocity="0.5" />
+        <origin xyz="0.0 0.0 0.0" />
+        <axis xyz="0.0 1.0 0.0" />
+        <limit effort="1000.0" lower="${Sternoklavikularjoint_posteriorrotation}" upper="${Sternoklavikularjoint_anteriorrotation}" velocity="0.5" />
     </xacro:joint_template>
 </robot>
