Commit message: added movement about the hips to the urdf model

File: ros2_ws/src/human_arm_model/urdf/alt_model.urdf.xacro (robot description, xacro)
@@ -17,24 +17,5 @@
         <!-- <xacro:minimal_interia /> -->
     </link>
-    <link name="columna"> <!-- carla columna-->
-        <visual>
-            <geometry>
-                <box size="${sternum_radius*2} ${sternum_radius*2} ${2*waist_back_length}"/>
-            </geometry>
-            <origin xyz="0.0 0.0 ${waist_back_length}"/>
-        </visual>
-        <collision>
-            <geometry>
-                <box size="${sternum_radius*2} ${sternum_radius*2} ${2*waist_back_length}"/>
-            </geometry>
-            <origin xyz="0.0 0.0 ${waist_back_length}"/>
-        </collision>
-        <xacro:box_inertia m="50.0" x="${sternum_radius*2}" y="${sternum_radius*2}" z="${2*waist_back_length}" />
-    </link>
-    <joint name="world_to_columna" type="fixed">
-        <parent link="base_link"/>
-        <child link="columna"/>
-        <origin xyz="0.0 0.0 0.0"/>
-    </joint>
+    <xacro:include filename="model2_folder/columna.urdf.xacro"/>
     <!-- placeholder mass here -->
     <xacro:cylinder_link_template name="clavicular" mass="1" radius="${sternum_radius/2}" height="${clavicle_link_length}">

File: ros2_ws/src/human_arm_model/urdf/model2_folder/sternoclavicular_joint.urdf.xacro (robot description, xacro)
@@ -9,6 +9,6 @@
         <xacro:minimal_interia />
     </link>
-    <xacro:joint_template bodypart="sternoclavicular" suffix="yaw" parent="columna" child="clavicular_yaw" >
-        <origin xyz="0.0 ${right * sternum_radius} ${2*waist_back_length}" rpy="0.0 0.0 ${right *30*math.pi/180}" />
+    <xacro:joint_template bodypart="sternoclavicular" suffix="yaw" parent="spine" child="clavicular_yaw" >
+        <origin xyz="0.0 ${right * sternum_radius} ${waist_back_length}" rpy="0.0 0.0 ${right *30*math.pi/180}" />
         <axis xyz="${right} 0.0 0.0" />
         <limit effort="1000.0" lower="${Sternoklavikularjoint_depression}" upper="${Sternoklavikularjoint_elevation}" velocity="0.5" />

Commit message: added origin of mass to URDF to use in Composite Rigid Body Algorithm

File: ros2_ws/src/human_arm_model/urdf/alt_model.urdf.xacro (robot description, xacro)
@@ -51,5 +51,7 @@
             <origin xyz="0.0 0.0 ${-hand_length/2}" rpy="${90*math.pi/180} 0.0 ${90*math.pi/180}"/>
         </collision>
-        <xacro:box_inertia m="${hand_weight}" x="${hand_thickness}" y="${hand_length}" z="${hand_width}" />
+        <xacro:box_inertia m="${hand_weight}" x="${hand_thickness}" y="${hand_length}" z="${hand_width}" >
+            <origin xyz="0.0 0.0 ${-hand_length/2}" rpy="${90*math.pi/180} 0.0 ${90*math.pi/180}"/>
+        </xacro:box_inertia>
     </link>
     <xacro:cylinder_link_template name="can" mass="${can_weight}" radius="${can_radius}" height="${can_height}">

File: ros2_ws/src/human_arm_model/urdf/macros.urdf.xacro (robot description, xacro)
@@ -29,15 +29,19 @@
                 </geometry>
             </collision>
-            <xacro:cylinder_inertia m="${mass}" r="${radius}" h="${height}"/>
+            <xacro:cylinder_inertia m="${mass}" r="${radius}" h="${height}">
+                <xacro:insert_block name="origin"/>
+            </xacro:cylinder_inertia>
         </link>
     </xacro:macro>
-    <xacro:macro name="cylinder_inertia" params="m r h">
+    <xacro:macro name="cylinder_inertia" params="m r h *origin">
         <inertial>
+            <xacro:insert_block name="origin"/>
             <mass value="${m}"/>
             <inertia ixx="${(1/12)* m*(3*r*r + h*h) }" ixy="0.0" ixz="0.0" iyy="${(1/12)* m*(3*r*r + h*h) }" iyz="0.0" izz="${(1/2)*m*r*r}" />
         </inertial>
     </xacro:macro>
-    <xacro:macro name="box_inertia" params="m x y z">
+    <xacro:macro name="box_inertia" params="m x y z *origin">
         <inertial>
+            <xacro:insert_block name="origin"/>
             <mass value="${m}"/>
             <inertia ixx="${(1/12)* m*(y*y + z*z) }" ixy="0.0" ixz="0.0" iyy="${(1/12)* m*(x*x + z*z) }" iyz="0.0" izz="${(1/12)*m* (x*x + y*y)}" />

File: ros2_ws/src/human_arm_model/urdf/model2_folder/columna.urdf.xacro (robot description, xacro)
@@ -17,5 +17,7 @@
             <origin xyz="0.0 0.0 ${waist_back_length/2}"/>
         </collision>
-        <xacro:box_inertia m="50.0" x="${sternum_radius}" y="${sternum_radius}" z="${waist_back_length}" />
+        <xacro:box_inertia m="50.0" x="${sternum_radius}" y="${sternum_radius}" z="${waist_back_length}" >
+            <origin xyz="0.0 0.0 ${waist_back_length/2}"/>
+        </xacro:box_inertia>
     </link>
     <joint name="world_to_columna" type="fixed">
@@ -37,5 +39,7 @@
             <origin xyz="0.0 0.0 ${waist_back_length/2}"/>
         </collision>
-        <xacro:box_inertia m="50.0" x="${sternum_radius}" y="${sternum_radius}" z="${waist_back_length}" />
+        <xacro:box_inertia m="50.0" x="${sternum_radius}" y="${sternum_radius}" z="${waist_back_length}">
+            <origin xyz="0.0 0.0 ${waist_back_length/2}"/>
+        </xacro:box_inertia>
     </link>
     <!-- forward tilt of 30° seems reasonable -->

Commit message: inertial origins now without rpy as needed for rbdl

File: ros2_ws/src/human_arm_model/urdf/alt_model.urdf.xacro (robot description, xacro)
@@ -19,11 +19,11 @@
     <xacro:include filename="model2_folder/columna.urdf.xacro"/>
     <!-- placeholder mass here -->
-    <xacro:cylinder_link_template name="clavicular" mass="1" radius="${sternum_radius/2}" height="${clavicle_link_length}">
+    <xacro:cylinder_link_template name="clavicular" mass="1" radius="${sternum_radius/2}" height="${clavicle_link_length}" dir_y="1.0" dir_z="0.0">
         <origin xyz="0.0 ${right * clavicle_link_length/2} 0.0" rpy="${math.pi/2} 0.0 0.0"/>
     </xacro:cylinder_link_template>
-    <xacro:cylinder_link_template name="humerus" mass="${upperarm_weight}" radius="${upperarm_radius}" height="${upperarm_length}">
+    <xacro:cylinder_link_template name="humerus" mass="${upperarm_weight}" radius="${upperarm_radius}" height="${upperarm_length}" dir_y="0.0" dir_z="1.0">
         <origin xyz="0.0 0.0 ${-upperarm_length/2}" rpy="0.0 0.0 0.0"/>
     </xacro:cylinder_link_template>
-    <xacro:cylinder_link_template name="forearm" mass="${forearm_weight}" radius="${forearm_circumference / (2*math.pi)}" height="${elbow_wrist_length}">
+    <xacro:cylinder_link_template name="forearm" mass="${forearm_weight}" radius="${forearm_circumference / (2*math.pi)}" height="${elbow_wrist_length}" dir_y="0.0" dir_z="1.0">
         <origin xyz="0.0 0.0 ${-elbow_wrist_length/2}" rpy="0.0 0.0 0.0"/>
     </xacro:cylinder_link_template>
@@ -52,8 +52,8 @@
         </collision>
         <xacro:box_inertia m="${hand_weight}" x="${hand_thickness}" y="${hand_length}" z="${hand_width}" >
-            <origin xyz="0.0 0.0 ${-hand_length/2}" rpy="${90*math.pi/180} 0.0 ${90*math.pi/180}"/>
+            <origin xyz="0.0 0.0 ${-hand_length/2}" rpy="0.0 0.0 0.0"/>
         </xacro:box_inertia>
     </link>
-    <xacro:cylinder_link_template name="can" mass="${can_weight}" radius="${can_radius}" height="${can_height}">
+    <xacro:cylinder_link_template name="can" mass="${can_weight}" radius="${can_radius}" height="${can_height}" dir_y="0.0" dir_z="0.0" dir_x="-1.0">
         <origin xyz="${-can_height/2} 0.0 0.0" rpy="${90*math.pi/180} 0.0 ${90*math.pi/180}"/>
     </xacro:cylinder_link_template>

File: ros2_ws/src/human_arm_model/urdf/macros.urdf.xacro (robot description, xacro)
@@ -15,5 +15,5 @@
         </joint>
     </xacro:macro>
-    <xacro:macro name="cylinder_link_template"  params="name mass radius height *origin ">
+    <xacro:macro name="cylinder_link_template"  params="name mass radius height dir_y dir_z dir_x:='0.0' *origin ">
         <link name="${name}">
             <visual>
@@ -29,12 +29,10 @@
                 </geometry>
             </collision>
-            <xacro:cylinder_inertia m="${mass}" r="${radius}" h="${height}">
-                <xacro:insert_block name="origin"/>
-            </xacro:cylinder_inertia>
+            <xacro:cylinder_inertia m="${mass}" r="${radius}" h="${height}" dir_y="${dir_y}" dir_z="${dir_z}" dir_x="${dir_x}"/>
         </link>
     </xacro:macro>
-    <xacro:macro name="cylinder_inertia" params="m r h *origin">
+    <xacro:macro name="cylinder_inertia" params="m r h dir_y dir_z dir_x">
         <inertial>
-            <xacro:insert_block name="origin"/>
+            <origin xyz="${dir_x * h/2.0} ${-1.0* dir_y*h/2.0} ${-1.0* dir_z*h/2.0}" rpy="0.0 0.0 0.0"/>
             <mass value="${m}"/>
             <inertia ixx="${(1/12)* m*(3*r*r + h*h) }" ixy="0.0" ixz="0.0" iyy="${(1/12)* m*(3*r*r + h*h) }" iyz="0.0" izz="${(1/2)*m*r*r}" />

Commit message: diverse

File: ros2_ws/src/human_arm_model/urdf/alt_model.urdf.xacro (robot description, xacro)
@@ -19,5 +19,5 @@
     <xacro:include filename="model2_folder/columna.urdf.xacro"/>
     <!-- placeholder mass here -->
-    <xacro:cylinder_link_template name="clavicular" mass="1" radius="${sternum_radius/2}" height="${clavicle_link_length}" dir_y="1.0" dir_z="0.0">
+    <xacro:cylinder_link_template name="clavicular" mass="3" radius="${clavicle_raidus}" height="${clavicle_link_length}" dir_y="1.0" dir_z="0.0">
         <origin xyz="0.0 ${right * clavicle_link_length/2} 0.0" rpy="${math.pi/2} 0.0 0.0"/>
     </xacro:cylinder_link_template>

File: ros2_ws/src/human_arm_model/urdf/constants.urdf.xacro (robot description, xacro)
@@ -19,4 +19,5 @@
     <xacro:property name="clavicle_link_length" value="0.2081" />
     <xacro:property name="sternum_radius" value="${clavicle_link_length - shoulder_length}" />
+    <xacro:property name="clavicle_raidus" value="0.015"/>
     <!-- Winkel -->
     <!-- Diese sind Bewegungsamplituden und nicht 1:1 im Model vorwendbar. -->

File: ros2_ws/src/human_arm_model/urdf/model2_folder/columna.urdf.xacro (robot description, xacro)
@@ -17,5 +17,5 @@
             <origin xyz="0.0 0.0 ${waist_back_length/2}"/>
         </collision>
-        <xacro:box_inertia m="50.0" x="${sternum_radius}" y="${sternum_radius}" z="${waist_back_length}" >
+        <xacro:box_inertia m="45.0" x="${sternum_radius}" y="${sternum_radius}" z="${waist_back_length}" >
             <origin xyz="0.0 0.0 ${waist_back_length/2}"/>
         </xacro:box_inertia>
@@ -39,5 +39,5 @@
             <origin xyz="0.0 0.0 ${waist_back_length/2}"/>
         </collision>
-        <xacro:box_inertia m="50.0" x="${sternum_radius}" y="${sternum_radius}" z="${waist_back_length}">
+        <xacro:box_inertia m="45.0" x="${sternum_radius}" y="${sternum_radius}" z="${waist_back_length}">
             <origin xyz="0.0 0.0 ${waist_back_length/2}"/>
         </xacro:box_inertia>

File: ros2_ws/src/human_arm_model/urdf/model3_folder/macros2.urdf.xacro (robot description, xacro)
@@ -13,5 +13,5 @@
     </xacro:macro>
     <!-- Inertia for a cylinder  -->
-    <xacro:macro name="cylinder_inertia" params="m r h">
+    <xacro:macro name="cylinder_inertia2" params="m r h">
         <inertial>
             <mass value="${m}"/>
@@ -51,5 +51,5 @@
                 </geometry>
             </collision>
-            <xacro:cylinder_inertia m="${mass}" r="${radius}" h="${height}"/>
+            <xacro:cylinder_inertia2 m="${mass}" r="${radius}" h="${height}"/>
         </link>
     </xacro:macro>
