Commit message: edb. adjustment

File: ros2_ws/src/human_arm_model/urdf/model3_folder/endeffector.urdf.xacro (robot description, xacro)
@@ -29,5 +29,5 @@
         <parent link="${prefix}hand"/>
         <child link="${prefix}can"/>
-        <origin xyz="${-can_radius} ${can_height/2} ${-hand_length}"/>
+        <origin xyz="${-can_radius-(hand_thickness/2)} ${can_height/2} ${-hand_length}"/>
     </joint>
 </robot>
