Commit message: some restructuring for better namespace

File: ros2_ws/model3.urdf (robot description, URDF)
Before this commit: robot human_arm_model3, 3 links, 1 joints
Links:
- added link model1_right_can, mass 0.45; collision cylinder length=0.12 radius=0.035; visual cylinder length=0.12 radius=0.035
- added link model1_right_elbow_1, mass 0.01
- added link model1_right_forearm, mass 1.4586000000000001; collision cylinder length=0.2869 radius=0.049353947852796745; visual cylinder length=0.2869 radius=0.049353947852796745
- added link model1_right_hand, mass 0.6006; collision box size=0.01784999999999999 0.1165 0.0883; visual box size=0.01784999999999999 0.1165 0.0883
- added link model1_right_upperarm, mass 2.4882; collision cylinder length=0.3637 radius=0.05699338512120772; visual cylinder length=0.3637 radius=0.05699338512120772
- link model1_right_torso: mass None -> 0.6006; geometry collision box size=0.4162 0.25699338512120773 0.9552; visual box size=0.4162 0.25699338512120773 0.9552
Joints:
- removed joint model1_right_shoulder_yaw_joint
- added joint model1_right_elbow_flexion_joint: type revolute, parent model1_right_upperarm, child model1_right_elbow_1, origin xyz=0.0 0.0 -0.3637, axis 1.0 0.0 0.0, limit lower=-0.2617993877991494 upper=2.792526803190927 effort=1000.0 velocity=0.5
- added joint model1_right_elbow_rotation_joint: type revolute, parent model1_right_elbow_1, child model1_right_forearm, origin xyz=0.0 0.0 0.0, axis 0.0 0.0 1.0, limit lower=-1.5707963267948966 upper=1.4835298641951802 effort=1000.0 velocity=0.5
- added joint model1_right_hand_can_joint: type fixed, parent model1_right_hand, child model1_right_can, origin xyz=0.0 -0.01784999999999999 -0.1165
- added joint model1_right_shoulder_abduction_joint: type revolute, parent model1_right_shoulder_1, child model1_right_shoulder_2, origin xyz=0.0 0.0 0.0, axis 0.0 -1.0 0.0, limit lower=-0.17453292519943295 upper=2.9670597283903604 effort=1000.0 velocity=0.5
- added joint model1_right_shoulder_flexion_joint: type revolute, parent model1_right_shoulder_2, child model1_right_upperarm, origin xyz=0.0 0.0 0.0, axis 1.0 0.0 0.0, limit lower=-1.0471975511965976 upper=2.9670597283903604 effort=1000.0 velocity=0.5
- added joint model1_right_shoulder_rotation_joint: type revolute, parent model1_right_torso, child model1_right_shoulder_1, origin xyz=0.2081 0.0 0.9552 rpy=0.0 0.0 0.0, axis 0.0 0.0 1.0, limit lower=-1.7453292519943295 upper=1.0471975511965976 effort=1000.0 velocity=0.5
- added joint model1_right_wrist_flexion_joint: type revolute, parent model1_right_forearm, child model1_right_hand, origin xyz=0.0 0.0 -0.2869, axis 0.0 1.0 0.0, limit lower=-1.4835298641951802 upper=1.4835298641951802 effort=1000.0 velocity=0.5

File: ros2_ws/src/human_arm_model/urdf/alt_model.urdf.xacro (robot description, xacro)
@@ -75,7 +75,7 @@
         <origin xyz="0.0 ${-hand_thickness} ${-hand_length} "/>
     </joint>
-    <xacro:include filename="alt_folder/sternoclavicular_joint.urdf.xacro" />
-    <xacro:include filename="alt_folder/glenohumeral_joint.urdf.xacro" />
-    <xacro:include filename="alt_folder/humeroulnar_joint.urdf.xacro" />
-    <xacro:include filename="alt_folder/alt_gazebo.urdf.xacro" />
+    <xacro:include filename="model2_folder/sternoclavicular_joint.urdf.xacro" />
+    <xacro:include filename="model2_folder/glenohumeral_joint.urdf.xacro" />
+    <xacro:include filename="model2_folder/humeroulnar_joint.urdf.xacro" />
+    <xacro:include filename="model2_folder/alt_gazebo.urdf.xacro" />
 </robot>

File: ros2_ws/src/human_arm_model/urdf/model3.urdf.xacro (robot description, xacro)
@@ -1,5 +1,5 @@
 <?xml version="1.0"?>
 <robot xmlns:xacro="http://www.ros.org/wiki/xacro" name="human_arm_model3">
-    <xacro:include filename="model_folder/macros2.urdf.xacro"/>
+    <xacro:include filename="model3_folder/macros2.urdf.xacro"/>
     <xacro:include filename="$(find human_arm_model)/urdf/constants.urdf.xacro" />
     <link name="${prefix}torso">
@@ -11,13 +11,21 @@
             <origin xyz="0.0 0.0 ${waist_back_length}"/>
         </visual>
+        <collision>
+            <geometry>
+                <!-- Bullshit limit for now  -->
+                <box size="${2*clavicle_link_length} ${0.2+ upperarm_circumference/ (2* math.pi)} ${2*waist_back_length}"/>
+            </geometry>
+            <origin xyz="0.0 0.0 ${waist_back_length}"/>
+        </collision>
+        <xacro:box_inertia m="${hand_weight}" x="${2*clavicle_link_length}" y="${0.2+ upperarm_circumference/ (2* math.pi)}" z="${2*waist_back_length}" />
     </link>
     <xacro:cylinder_link_template2 name="upperarm" mass="${upperarm_weight}" radius="${upperarm_radius}" height="${upperarm_length}">
         <origin xyz="0.0 0.0 ${-upperarm_length/2}" rpy="0.0 0.0 0.0"/>
     </xacro:cylinder_link_template2>
-    <xacro:include filename="model_folder/shoulder.urdf.xacro"/>
+    <xacro:include filename="model3_folder/shoulder.urdf.xacro"/>
     <xacro:cylinder_link_template2 name="forearm" mass="${forearm_weight}" radius="${forearm_circumference / (2*math.pi)}" height="${elbow_wrist_length}">
         <origin xyz="0.0 0.0 ${-elbow_wrist_length/2}" rpy="0.0 0.0 0.0"/>
     </xacro:cylinder_link_template2>
-    <xacro:include filename="model_folder/elbow.urdf.xacro"/>
-    <xacro:include filename="model_folder/endeffector.urdf.xacro"/>
+    <xacro:include filename="model3_folder/elbow.urdf.xacro"/>
+    <xacro:include filename="model3_folder/endeffector.urdf.xacro"/>
 </robot>

File: ros2_ws/src/human_arm_model/urdf/model3_folder/elbow.urdf.xacro (robot description, xacro)
@@ -2,5 +2,5 @@
 <robot xmlns:xacro="http://www.ros.org/wiki/xacro" name="human_arm_model">
     <xacro:include filename="$(find human_arm_model)/urdf/constants.urdf.xacro" />
-    <xacro:include filename="macros.urdf.xacro" />
+    <xacro:include filename="macros2.urdf.xacro" />
     <link name="${prefix}elbow_1">
         <xacro:minimal_inertia />

File: ros2_ws/src/human_arm_model/urdf/model3_folder/endeffector.urdf.xacro (robot description, xacro)
@@ -2,5 +2,5 @@
 <robot xmlns:xacro="http://www.ros.org/wiki/xacro" name="human_arm_model">
     <xacro:include filename="$(find human_arm_model)/urdf/constants.urdf.xacro" />
-    <xacro:include filename="macros.urdf.xacro" />
+    <xacro:include filename="macros2.urdf.xacro" />
     <link name="${prefix}hand">
         <visual>

File: ros2_ws/src/human_arm_model/urdf/model3_folder/shoulder.urdf.xacro (robot description, xacro)
@@ -2,5 +2,5 @@
 <robot xmlns:xacro="http://www.ros.org/wiki/xacro" name="human_arm_model">
     <xacro:include filename="$(find human_arm_model)/urdf/constants.urdf.xacro" />
-    <xacro:include filename="macros.urdf.xacro" />
+    <xacro:include filename="macros2.urdf.xacro" />
     <link name="${prefix}shoulder_1">
         <xacro:minimal_inertia />

Commit message: collision checking fixed

File: ros2_ws/model3.urdf (robot description, URDF)
Before this commit: robot human_arm_model3, 8 links, 7 joints
Joints:
- joint model1_right_hand_can_joint: origin xyz=0.0 -0.01784999999999999 -0.1165 -> xyz=0.0 0.0 -0.1165

File: ros2_ws/src/human_arm_model/urdf/model3_folder/endeffector.urdf.xacro (robot description, xacro)
@@ -29,5 +29,5 @@
         <parent link="${prefix}hand"/>
         <child link="${prefix}can"/>
-        <origin xyz="0.0 ${-hand_thickness} ${-hand_length}"/>
+        <origin xyz="0.0 0.0 ${-hand_length}"/>
     </joint>
 </robot>

Commit message: changes to model according to warn messages from rviz

File: ros2_ws/model3.urdf (robot description, URDF)
Before this commit: robot human_arm_model3, 8 links, 7 joints
Links:
- link model1_right_torso: mass 0.6006 -> None

File: ros2_ws/src/human_arm_model/urdf/model3.urdf.xacro (robot description, xacro)
@@ -18,5 +18,5 @@
             <origin xyz="0.0 0.0 ${waist_back_length}"/>
         </collision>
-        <xacro:box_inertia m="${hand_weight}" x="${2*clavicle_link_length}" y="${0.2+ upperarm_circumference/ (2* math.pi)}" z="${2*waist_back_length}" />
+        <!-- <xacro:box_inertia m="${hand_weight}" x="${2*clavicle_link_length}" y="${0.2+ upperarm_circumference/ (2* math.pi)}" z="${2*waist_back_length}" /> -->
     </link>
     <xacro:cylinder_link_template2 name="upperarm" mass="${upperarm_weight}" radius="${upperarm_radius}" height="${upperarm_length}">

Commit message: can's TF coordinates are now positioned at the same place the datapoints are taken

File: ros2_ws/model3.urdf (robot description, URDF)
Before this commit: robot human_arm_model3, 8 links, 7 joints
Joints:
- joint model1_right_hand_can_joint: origin xyz=0.0 0.0 -0.1165 -> xyz=-0.035 0.06 -0.1165

File: ros2_ws/src/human_arm_model/urdf/model3_folder/endeffector.urdf.xacro (robot description, xacro)
@@ -24,10 +24,10 @@
     </xacro:joint_template2>
     <xacro:cylinder_link_template2 name="can" mass="${can_weight}" radius="${can_radius}" height="${can_height}">
-        <origin xyz="${-can_radius} 0.0 0.0" rpy="${90*math.pi/180} 0.0 0.0"/>
+        <origin xyz="0.0 ${-can_height/2} 0.0" rpy="${90*math.pi/180} 0.0 0.0"/>
     </xacro:cylinder_link_template2>
     <joint name="${prefix}hand_can_joint" type="fixed">
         <parent link="${prefix}hand"/>
         <child link="${prefix}can"/>
-        <origin xyz="0.0 0.0 ${-hand_length}"/>
+        <origin xyz="${-can_radius} ${can_height/2} ${-hand_length}"/>
     </joint>
 </robot>

Commit message: after reaching the first position first implementation try for path following

File: ros2_ws/model3.urdf (robot description, URDF)
Before this commit: robot human_arm_model3, 8 links, 7 joints
Joints:
- joint model1_right_hand_can_joint: origin xyz=-0.035 0.06 -0.1165 -> xyz=-0.043925 0.06 -0.1165
