Commit message: alt_model now fit for usage with sim. -> can is now center of calculations

File: ros2_ws/alt_model.urdf (robot description, URDF)
Before this commit: robot alt_human_arm_model, 12 links, 11 joints
Links:
- link columna: mass 50 -> 50.0
Joints:
- joint elbow_roll_joint: axis 0 0 1 -> 0.0 0.0 1.0; limit lower=-1.5707963267948966 upper=1.4835298641951802 effort=1000 velocity=0.5 -> lower=-1.5707963267948966 upper=1.4835298641951802 effort=1000.0 velocity=0.5; origin xyz=0 0 0 -> xyz=0.0 0.0 0.0
- joint elbow_yaw_joint: axis 0 -1 0 -> 0.0 -1.0 0.0; limit lower=-0.2617993877991494 upper=2.792526803190927 effort=1000 velocity=0.5 -> lower=-0.2617993877991494 upper=2.792526803190927 effort=1000.0 velocity=0.5; origin xyz=0 0 -0.3637 -> xyz=0.0 0.0 -0.3637
- joint glenohumeral_pitch_joint: axis 0 -1 0 -> 0.0 -1.0 0.0; limit lower=-0.6981317007977318 upper=1.3962634015954636 effort=1000 velocity=0.5 -> lower=-0.6981317007977318 upper=1.3962634015954636 effort=1000.0 velocity=0.5; origin xyz=0 0 0 -> xyz=0.0 0.0 0.0
- joint glenohumeral_roll_joint: axis 0 0 1 -> 0.0 0.0 1.0; limit lower=-1.7453292519943295 upper=1.0471975511965976 effort=1000 velocity=0.5 -> lower=-1.7453292519943295 upper=1.0471975511965976 effort=1000.0 velocity=0.5; origin xyz=0 0 0 -> xyz=0.0 0.0 0.0
- joint glenohumeral_yaw_joint: axis 1 0 0 -> 1.0 0.0 0.0; limit lower=0.0 upper=1.5707963267948966 effort=1000 velocity=0.5 -> lower=0.0 upper=1.5707963267948966 effort=1000.0 velocity=0.5; origin xyz=0 0.2081 0 rpy=0 0 -0.5235987755982988 -> xyz=0.0 0.2081 0.0 rpy=0.0 0.0 -0.5235987755982988
- joint hand_can_joint: origin xyz=0 -0.01784999999999999 -0.1165  -> xyz=0.06 -0.043925 -0.1165
- joint sternoclavicular_pitch_joint: axis 0 0 1 -> 0.0 0.0 1.0; limit lower=-0.5235987755982988 upper=0.5235987755982988 effort=1000 velocity=0.5 -> lower=-0.5235987755982988 upper=0.5235987755982988 effort=1000.0 velocity=0.5; origin xyz=0 0 0 -> xyz=0.0 0.0 0.0
- joint sternoclavicular_roll_joint: axis 0 1 0 -> 0.0 1.0 0.0; limit lower=-0.5235987755982988 upper=0.5235987755982988 effort=1000 velocity=0.5 -> lower=-0.5235987755982988 upper=0.5235987755982988 effort=1000.0 velocity=0.5; origin xyz=0 0 0 -> xyz=0.0 0.0 0.0
- joint sternoclavicular_yaw_joint: axis 1 0 0 -> 1.0 0.0 0.0; limit lower=-0.08726646259971647 upper=0.5235987755982988 effort=1000 velocity=0.5 -> lower=-0.08726646259971647 upper=0.5235987755982988 effort=1000.0 velocity=0.5; origin xyz=0 0.05830000000000002 0.9552 rpy=0 0 0.5235987755982988 -> xyz=0.0 0.05830000000000002 0.9552 rpy=0.0 0.0 0.5235987755982988
- joint world_to_columna: origin xyz=0 0 0 -> xyz=0.0 0.0 0.0
- joint wrist_yaw_joint: axis 1 0 0 -> 1.0 0.0 0.0; limit lower=-1.4835298641951802 upper=1.4835298641951802 effort=1000 velocity=0.5 -> lower=-1.4835298641951802 upper=1.4835298641951802 effort=1000.0 velocity=0.5; origin xyz=0 0 -0.2869 -> xyz=0.0 0.0 -0.2869

File: ros2_ws/src/human_arm_model/urdf/alt_model.urdf.xacro (robot description, xacro)
@@ -68,14 +68,14 @@
     </link>
     <xacro:cylinder_link_template name="can" mass="${can_weight}" radius="${can_radius}" height="${can_height}">
-        <origin xyz="0.0 0.0 0.0" rpy="${90*math.pi/180} 0.0 ${90*math.pi/180}"/>
+        <origin xyz="${-can_height/2} 0.0 0.0" rpy="${90*math.pi/180} 0.0 ${90*math.pi/180}"/>
     </xacro:cylinder_link_template>
     <joint name="hand_can_joint" type="fixed">
         <parent link="hand"/>
         <child link="can"/>
-        <origin xyz="0.0 ${-hand_thickness} ${-hand_length} "/>
+        <origin xyz="${can_height/2} ${-(hand_thickness/2) - can_radius } ${-hand_length}"/>
     </joint>
     <xacro:include filename="model2_folder/sternoclavicular_joint.urdf.xacro" />
     <xacro:include filename="model2_folder/glenohumeral_joint.urdf.xacro" />
     <xacro:include filename="model2_folder/humeroulnar_joint.urdf.xacro" />
-    <xacro:include filename="model2_folder/alt_gazebo.urdf.xacro" />
+    <!-- <xacro:include filename="model2_folder/alt_gazebo.urdf.xacro" /> -->
 </robot>

Commit message: wrist is now fixed and no longer controllable in model

File: ros2_ws/alt_model.urdf (robot description, URDF)
Before this commit: robot alt_human_arm_model, 12 links, 11 joints
Joints:
- removed joint wrist_yaw_joint
- added joint forearm_hand_joint: type fixed, parent forearm, child hand, origin xyz=0.0 0.0 -0.2869

File: ros2_ws/src/human_arm_model/urdf/alt_model.urdf.xacro (robot description, xacro)
@@ -47,9 +47,14 @@
         <origin xyz="0.0 0.0 ${-elbow_wrist_length/2}" rpy="0.0 0.0 0.0"/>
     </xacro:cylinder_link_template>
-    <xacro:bodypart_template bodypart="wrist" suffix="yaw" parent="forearm" child="hand">
+    <!-- <xacro:bodypart_template bodypart="wrist" suffix="yaw" parent="forearm" child="hand">
         <origin xyz="0.0 0.0 ${-elbow_wrist_length}"/>
         <axis xyz="1.0 0.0 0.0" />
         <limit effort="1000.0" lower="${hand_palmarflexion}" upper="${hand_dorsalextension}" velocity="0.5" />
-    </xacro:bodypart_template>
+    </xacro:bodypart_template> -->
+    <joint name="forearm_hand_joint" type="fixed">
+        <parent link="forearm"/>
+        <child link="hand"/>
+        <origin xyz="0.0 0.0 ${-elbow_wrist_length}"/>
+    </joint>
     <link name="hand">
         <visual>

File: ros2_ws/src/human_arm_model/urdf/constants.urdf.xacro (robot description, xacro)
@@ -59,3 +59,4 @@
     <xacro:property name="hand_weight" value="${bodyweight * 0.007}" />
     <xacro:property name="can_weight" value="0.45"/>
+    <xacro:arg name="side" default="right"/>
 </robot>

File: ros2_ws/src/moveit_config/config/alt_human_arm_model.ros2_control.xacro (robot description, xacro)
@@ -64,5 +64,5 @@
                 <state_interface name="velocity"/>
             </joint>
-            <joint name="wrist_yaw_joint">
+            <!-- <joint name="wrist_yaw_joint">
                 <command_interface name="position"/>
                 <state_interface name="position">
@@ -70,5 +70,5 @@
                 </state_interface>
                 <state_interface name="velocity"/>
-            </joint>
+            </joint> -->
         </ros2_control>
     </xacro:macro>

Commit message: model now uses right hand per default, not left hand; Pos1 as default position is invalidated

File: ros2_ws/alt_model.urdf (robot description, URDF)
Before this commit: robot alt_human_arm_model, 12 links, 11 joints
Joints:
- joint glenohumeral_yaw_joint: axis 1.0 0.0 0.0 -> -1 0.0 0.0; origin xyz=0.0 0.2081 0.0 rpy=0.0 0.0 -0.5235987755982988 -> xyz=0.0 -0.2081 0.0 rpy=0.0 0.0 -0.5235987755982988
- joint hand_can_joint: origin xyz=0.06 -0.043925 -0.1165 -> xyz=0.06 0.043925 -0.1165
- joint sternoclavicular_yaw_joint: axis 1.0 0.0 0.0 -> -1 0.0 0.0; origin xyz=0.0 0.05830000000000002 0.9552 rpy=0.0 0.0 0.5235987755982988 -> xyz=0.0 -0.05830000000000002 0.9552 rpy=0.0 0.0 0.5235987755982988

File: ros2_ws/src/human_arm_model/urdf/alt_model.urdf.xacro (robot description, xacro)
@@ -39,5 +39,5 @@
     <!-- placeholder mass here -->
     <xacro:cylinder_link_template name="clavicular" mass="1" radius="${sternum_radius/2}" height="${clavicle_link_length}">
-        <origin xyz="0.0 ${clavicle_link_length/2} 0.0" rpy="${math.pi/2} 0.0 0.0"/>
+        <origin xyz="0.0 ${right * clavicle_link_length/2} 0.0" rpy="${math.pi/2} 0.0 0.0"/>
     </xacro:cylinder_link_template>
     <xacro:cylinder_link_template name="humerus" mass="${upperarm_weight}" radius="${upperarm_radius}" height="${upperarm_length}">
@@ -78,5 +78,5 @@
         <parent link="hand"/>
         <child link="can"/>
-        <origin xyz="${can_height/2} ${-(hand_thickness/2) - can_radius } ${-hand_length}"/>
+        <origin xyz="${can_height/2} ${right * (-(hand_thickness/2) - can_radius) } ${-hand_length}"/>
     </joint>
     <xacro:include filename="model2_folder/sternoclavicular_joint.urdf.xacro" />

File: ros2_ws/src/human_arm_model/urdf/constants.urdf.xacro (robot description, xacro)
@@ -60,3 +60,9 @@
     <xacro:property name="can_weight" value="0.45"/>
     <xacro:arg name="side" default="right"/>
+    <xacro:if value="${'$(arg side)'=='right'}">
+        <xacro:property name="right" value="-1"/>
+    </xacro:if>
+    <xacro:unless value="${'$(arg side)'=='right'}">
+        <xacro:property name="right" value="1"/>
+    </xacro:unless>
 </robot>

File: ros2_ws/src/human_arm_model/urdf/model2_folder/glenohumeral_joint.urdf.xacro (robot description, xacro)
@@ -10,6 +10,6 @@
     </link>
     <xacro:joint_template bodypart="glenohumeral" suffix="yaw" parent="clavicular" child="humerus_yaw" >
-        <origin xyz="0.0 ${clavicle_link_length} 0.0" rpy="0.0 0.0 ${-30*math.pi/180}"/>
-        <axis xyz="1.0 0.0 0.0" />
+        <origin xyz="0.0 ${right * clavicle_link_length} 0.0" rpy="0.0 0.0 ${-30*math.pi/180}"/>
+        <axis xyz="${right} 0.0 0.0" />
         <limit effort="1000.0" lower="${glenohumeraljoint_adduktion}" upper="${glenohumeraljoint_abduktion}" velocity="0.5" />
     </xacro:joint_template>

File: ros2_ws/src/human_arm_model/urdf/model2_folder/sternoclavicular_joint.urdf.xacro (robot description, xacro)
@@ -10,6 +10,6 @@
     </link>
     <xacro:joint_template bodypart="sternoclavicular" suffix="yaw" parent="columna" child="clavicular_yaw" >
-        <origin xyz="0.0 ${sternum_radius} ${2*waist_back_length}" rpy="0.0 0.0 ${30*math.pi/180}" />
-        <axis xyz="1.0 0.0 0.0" />
+        <origin xyz="0.0 ${right * sternum_radius} ${2*waist_back_length}" rpy="0.0 0.0 ${30*math.pi/180}" />
+        <axis xyz="${right} 0.0 0.0" />
         <limit effort="1000.0" lower="${Sternoklavikularjoint_depression}" upper="${Sternoklavikularjoint_elevation}" velocity="0.5" />
     </xacro:joint_template>

Commit message: fixed issue in right arm where clavicula would be oriented in the wrong direction

File: ros2_ws/alt_model.urdf (robot description, URDF)
Before this commit: robot alt_human_arm_model, 12 links, 11 joints
Joints:
- joint glenohumeral_yaw_joint: origin xyz=0.0 -0.2081 0.0 rpy=0.0 0.0 -0.5235987755982988 -> xyz=0.0 -0.2081 0.0 rpy=0.0 0.0 0.5235987755982988
- joint sternoclavicular_yaw_joint: origin xyz=0.0 -0.05830000000000002 0.9552 rpy=0.0 0.0 0.5235987755982988 -> xyz=0.0 -0.05830000000000002 0.9552 rpy=0.0 0.0 -0.5235987755982988

File: ros2_ws/src/human_arm_model/urdf/model2_folder/glenohumeral_joint.urdf.xacro (robot description, xacro)
@@ -10,5 +10,5 @@
     </link>
     <xacro:joint_template bodypart="glenohumeral" suffix="yaw" parent="clavicular" child="humerus_yaw" >
-        <origin xyz="0.0 ${right * clavicle_link_length} 0.0" rpy="0.0 0.0 ${-30*math.pi/180}"/>
+        <origin xyz="0.0 ${right * clavicle_link_length} 0.0" rpy="0.0 0.0 ${right * -30*math.pi/180}"/>
         <axis xyz="${right} 0.0 0.0" />
         <limit effort="1000.0" lower="${glenohumeraljoint_adduktion}" upper="${glenohumeraljoint_abduktion}" velocity="0.5" />

File: ros2_ws/src/human_arm_model/urdf/model2_folder/sternoclavicular_joint.urdf.xacro (robot description, xacro)
@@ -10,5 +10,5 @@
     </link>
     <xacro:joint_template bodypart="sternoclavicular" suffix="yaw" parent="columna" child="clavicular_yaw" >
-        <origin xyz="0.0 ${right * sternum_radius} ${2*waist_back_length}" rpy="0.0 0.0 ${30*math.pi/180}" />
+        <origin xyz="0.0 ${right * sternum_radius} ${2*waist_back_length}" rpy="0.0 0.0 ${right *30*math.pi/180}" />
         <axis xyz="${right} 0.0 0.0" />
         <limit effort="1000.0" lower="${Sternoklavikularjoint_depression}" upper="${Sternoklavikularjoint_elevation}" velocity="0.5" />

Commit message: moveit now uses the new joint about the hips

File: ros2_ws/alt_model.urdf (robot description, URDF)
Before this commit: robot alt_human_arm_model, 12 links, 11 joints
Links:
- added link spine, mass 50.0; collision box size=0.11660000000000004 0.11660000000000004 0.4776; visual box size=0.11660000000000004 0.11660000000000004 0.4776
- link columna: geometry collision box size=0.11660000000000004 0.11660000000000004 0.4776; visual box size=0.11660000000000004 0.11660000000000004 0.4776
Joints:
- added joint columna__joint: type revolute, parent columna, child spine, origin xyz=0.0 0.0 0.4776 rpy=0.0 0.0 0.0, axis 0.0 1.0 0.0, limit lower=0.0 upper=0.5235987755982988 effort=1000.0 velocity=0.5
- joint sternoclavicular_yaw_joint: origin xyz=0.0 -0.05830000000000002 0.9552 rpy=0.0 0.0 -0.5235987755982988 -> xyz=0.0 -0.05830000000000002 0.4776 rpy=0.0 0.0 -0.5235987755982988; parent columna -> spine

File: ros2_ws/src/moveit_config/config/alt_human_arm_model.ros2_control.xacro (robot description, xacro)
@@ -8,4 +8,11 @@
                 <plugin>mock_components/GenericSystem</plugin>
             </hardware>
+            <joint name="columna__joint">
+                <command_interface name="position"/>
+                <state_interface name="position">
+                  <param name="initial_value">${initial_positions['columna__joint']}</param>
+                </state_interface>
+                <state_interface name="velocity"/>
+            </joint>
             <joint name="sternoclavicular_yaw_joint">
                 <command_interface name="position"/>

Commit message: WIP using custom cost fn backwards movement

File: ros2_ws/alt_model.urdf (robot description, URDF)
Before this commit: robot alt_human_arm_model, 13 links, 12 joints
Joints:
- joint columna__joint: limit lower=0.0 upper=0.5235987755982988 effort=1000.0 velocity=0.5 -> lower=0.0 upper=0.08726646259971647 effort=1000.0 velocity=0.5

File: ros2_ws/src/human_arm_model/urdf/model2_folder/columna.urdf.xacro (robot description, xacro)
@@ -43,5 +43,5 @@
         <origin xyz="0.0 0.0 ${waist_back_length}" rpy="0.0 0.0 0.0" />
         <axis xyz="0.0 1.0 0.0" />
-        <limit effort="1000.0" lower="0.0" upper="${30*math.pi/180}" velocity="0.5" />
+        <limit effort="1000.0" lower="0.0" upper="${5*math.pi/180}" velocity="0.5" />
     </xacro:joint_template>
 </robot>

Commit message: additional rotation in spine allows for more realistic movement (especially to the left)

File: ros2_ws/alt_model.urdf (robot description, URDF)
Before this commit: robot alt_human_arm_model, 13 links, 12 joints
Links:
- added link c1, mass 0.01
Joints:
- removed joint columna__joint
- added joint columna_flex_joint: type revolute, parent c1, child spine, origin xyz=0.0 0.0 0.0 rpy=0.0 0.0 0.0, axis 0.0 1.0 0.0, limit lower=0.0 upper=0.5235987755982988 effort=1000.0 velocity=0.5
- added joint columna_rot_joint: type revolute, parent columna, child c1, origin xyz=0.0 0.0 0.4776 rpy=0.0 0.0 0.0, axis 0.0 0.0 1.0, limit lower=-0.5235987755982988 upper=0.5235987755982988 effort=1000.0 velocity=0.5

File: ros2_ws/src/human_arm_model/urdf/model2_folder/columna.urdf.xacro (robot description, xacro)
@@ -40,8 +40,17 @@
     </link>
     <!-- forward tilt of 30° seems reasonable -->
-    <xacro:joint_template bodypart="columna" suffix="" parent="columna" child="spine" >
-        <origin xyz="0.0 0.0 ${waist_back_length}" rpy="0.0 0.0 0.0" />
+    <xacro:joint_template bodypart="columna" suffix="flex" parent="c1" child="spine" >
+        <origin xyz="0.0 0.0 0.0" rpy="0.0 0.0 0.0" />
         <axis xyz="0.0 1.0 0.0" />
         <limit effort="1000.0" lower="0.0" upper="${30*math.pi/180}" velocity="0.5" />
     </xacro:joint_template>
+    <link name="c1">
+        <xacro:minimal_interia />
+    </link>
+    <!-- rotation of 70-80° in each direction is possible, but 30° will sufice -->
+    <xacro:joint_template bodypart="columna" suffix="rot" parent="columna" child="c1">
+        <origin xyz="0.0 0.0 ${waist_back_length}" rpy="0.0 0.0 0.0" />
+        <axis xyz="0.0 0.0 1.0" />
+        <limit effort="1000.0" lower="${-30*math.pi/180}" upper="${30*math.pi/180}" velocity="0.5" />
+    </xacro:joint_template>
 </robot>

File: ros2_ws/src/moveit_config/config/alt_human_arm_model.ros2_control.xacro (robot description, xacro)
@@ -8,8 +8,15 @@
                 <plugin>mock_components/GenericSystem</plugin>
             </hardware>
-            <joint name="columna__joint">
+            <joint name="columna_rot_joint">
                 <command_interface name="position"/>
                 <state_interface name="position">
-                  <param name="initial_value">${initial_positions['columna__joint']}</param>
+                  <param name="initial_value">${initial_positions['columna_rot_joint']}</param>
+                </state_interface>
+                <state_interface name="velocity"/>
+            </joint>
+            <joint name="columna_flex_joint">
+                <command_interface name="position"/>
+                <state_interface name="position">
+                  <param name="initial_value">${initial_positions['columna_flex_joint']}</param>
                 </state_interface>
                 <state_interface name="velocity"/>

Commit message: rotation about the hips increased to lower bound of human capable movement

File: ros2_ws/alt_model.urdf (robot description, URDF)
Before this commit: robot alt_human_arm_model, 14 links, 13 joints
Joints:
- joint columna_rot_joint: limit lower=-0.5235987755982988 upper=0.5235987755982988 effort=1000.0 velocity=0.5 -> lower=-1.2217304763960306 upper=1.2217304763960306 effort=1000.0 velocity=0.5

File: ros2_ws/src/human_arm_model/urdf/model2_folder/columna.urdf.xacro (robot description, xacro)
@@ -48,9 +48,9 @@
         <xacro:minimal_interia />
     </link>
-    <!-- rotation of 70-80° in each direction is possible, but 30° will sufice -->
+    <!-- rotation of 70-80° in each direction is possible -->
     <xacro:joint_template bodypart="columna" suffix="rot" parent="columna" child="c1">
         <origin xyz="0.0 0.0 ${waist_back_length}" rpy="0.0 0.0 0.0" />
         <axis xyz="0.0 0.0 1.0" />
-        <limit effort="1000.0" lower="${-30*math.pi/180}" upper="${30*math.pi/180}" velocity="0.5" />
+        <limit effort="1000.0" lower="${-70*math.pi/180}" upper="${70*math.pi/180}" velocity="0.5" />
     </xacro:joint_template>
 </robot>
